Commit message: Fixing small mistakes

File: depthai_bridge/urdf/rae_gazebo.urdf.xacro (robot description, xacro)
@@ -4,5 +4,5 @@
     <link name="base_frame"/>
     <link name="chassis">
-      <xacro:body mass="0.5" d="0.125" h="0.028" w="0.1256">
+      <xacro:body mass="0.2" d="0.125" h="0.028" w="0.1256">
           <origin xyz="0 0.014 0.0" rpy="0.0 0.0 0.0"/>
       </xacro:body>
@@ -10,5 +10,5 @@
         <origin rpy="0.0 0.0 0.0" xyz="0.0 0.0 0.0"/>
         <geometry>
-          <mesh filename="package://depthai_bridge/urdf/models/RAE-enclosure_01051900.stl" scale="0.001 0.001 0.001"/>
+          <mesh filename="package://depthai_bridge/urdf/models/RAE.stl" scale="1.0 1.0 1.0"/>
         </geometry>
       </collision>
@@ -16,5 +16,5 @@
         <origin rpy="0.0 0.0 0.0" xyz="0.0 0.0 0.0"/>
         <geometry>
-          <mesh filename="package://depthai_bridge/urdf/models/RAE-enclosure_01051900.stl" scale="0.001 0.001 0.001"/>
+          <mesh filename="package://depthai_bridge/urdf/models/RAE.stl" scale="1.0 1.0 1.0"/>
         </geometry>
         <material name="mat">
@@ -40,5 +40,5 @@
         <origin rpy="0.0 0.0 0.0" xyz="-0.0125 0.0 0.0"/>
         <geometry>
-            <mesh filename="package://depthai_bridge/urdf/models/RAE-Wheel_01051900.stl" scale="0.001 0.001 0.001"/>
+            <mesh filename="package://depthai_bridge/urdf/models/Motor-wheel.stl" scale="1.0 1.0 1.0"/>
         </geometry>
       </collision>
@@ -46,5 +46,5 @@
         <origin rpy="0.0 0.0 0.0" xyz="-0.0125 0.0 0.0"/>
         <geometry>
-            <mesh filename="package://depthai_bridge/urdf/models/RAE-Wheel_01051900.stl" scale="0.001 0.001 0.001"/>
+            <mesh filename="package://depthai_bridge/urdf/models/Motor-wheel.stl" scale="1.0 1.0 1.0"/>
         </geometry>
       </visual>
@@ -57,5 +57,5 @@
         <origin rpy="0.0 0.0 0.0" xyz="-0.0125 0.0 0.0"/>
         <geometry>
-            <mesh filename="package://depthai_bridge/urdf/models/RAE-Wheel_01051900.stl" scale="0.001 0.001 0.001"/>
+            <mesh filename="package://depthai_bridge/urdf/models/Motor-wheel.stl" scale="1.0 1.0 1.0"/>
         </geometry>
       </collision>
@@ -63,5 +63,5 @@
         <origin rpy="0.0 0.0 0.0" xyz="-0.0125 0.0 0.0"/>
         <geometry>
-            <mesh filename="package://depthai_bridge/urdf/models/RAE-Wheel_01051900.stl" scale="0.001 0.001 0.001"/>
+            <mesh filename="package://depthai_bridge/urdf/models/Motor-wheel.stl" scale="1.0 1.0 1.0"/>
         </geometry>
       </visual>
@@ -80,5 +80,5 @@
     </joint>
     <link name="left_caster_wheel">
-      <xacro:caster_wheels mass="0.035" r="0.005">
+      <xacro:caster_wheels mass="0.05" r="0.005">
             <origin xyz="0.0 0.0 0.0" rpy="0.0 0.0 0.0"/>
       </xacro:caster_wheels>
@@ -118,5 +118,5 @@
     </joint>
     <link name="right_caster_wheel">
-      <xacro:caster_wheels mass="0.035" r="0.005">
+      <xacro:caster_wheels mass="0.05" r="0.005">
             <origin xyz="0.0 0.0 0.0" rpy="0.0 0.0 0.0"/>
       </xacro:caster_wheels>
