Commit message: Small updates to launch files and urdfs

File: rae_description/urdf/rae_gazebo.urdf.xacro (robot description, xacro)
@@ -7,5 +7,13 @@
      </xacro:body>
     </link>
-<link name="chassis">
+    <gazebo reference="base_frame">
+     <sensor name="imu_sensor" type="imu">
+      <always_on>1</always_on>
+      <update_rate>1</update_rate>
+      <visualize>true</visualize>
+      <topic>imu</topic>
+     </sensor>
+    </gazebo>
+    <link name="chassis">
       <xacro:body mass="0.2" d="0.125" h="0.028" w="0.1256">
           <origin xyz="0 0.014 0.0" rpy="0.0 0.0 0.0"/>

Commit message: adding depth and segmentation camera

File: rae_description/urdf/rae_gazebo.urdf.xacro (robot description, xacro)
@@ -100,12 +100,4 @@
           <mesh filename="package://rae_description/urdf/models/caster-wheel.stl" scale="1.0 1.0 1.0"/>
         </geometry>
-        <surface>
-          <friction>
-            <ode>
-              <mu>0.01</mu>
-              <mu2>0.01</mu2>
-            </ode>
-          </friction>
-        </surface>
       </collision>
       <visual>
@@ -138,12 +130,4 @@
           <mesh filename="package://rae_description/urdf/models/caster-wheel.stl" scale="1.0 1.0 1.0"/>
         </geometry>
-        <surface>
-          <friction>
-            <ode>
-              <mu>0.01</mu>
-              <mu2>0.01</mu2>
-            </ode>
-          </friction>
-        </surface>
       </collision>
       <visual>
@@ -205,8 +189,28 @@
      </xacro:body>
     </link>
+    <link name="segmentation_camera_link_optical_frame">
+     <xacro:body mass="0.00001" d="0.0000010" h="0.000003" w="0.00003">
+          <origin xyz="0.0 0.0 0.0" rpy="0.0 0.0 0.0"/>
+     </xacro:body>
+    </link>
+    <link name="depth_camera_link_optical_frame">
+     <xacro:body mass="0.00001" d="0.0000010" h="0.000003" w="0.00003">
+          <origin xyz="0.0 0.0 0.0" rpy="0.0 0.0 0.0"/>
+     </xacro:body>
+    </link>
     <joint name="rgb_camera_link_optical_frame_joint" type="fixed">
       <origin xyz="0.0051 0 0" rpy="-1.57 0.0 -1.57"/>
       <parent link="rgb_camera_link"/>
       <child link="rgb_camera_link_optical_frame"/>
+    </joint>
+    <joint name="segmentation_camera_link_optical_frame_joint" type="fixed">
+      <origin xyz="0.0051 0 0" rpy="0.0 0.0 0.0"/>
+      <parent link="rgb_camera_link"/>
+      <child link="segmentation_camera_link_optical_frame"/>
+    </joint>
+    <joint name="depth_camera_link_optical_frame_joint" type="fixed">
+      <origin xyz="0.0051 0 0" rpy="0.0 0.0 0.0"/>
+      <parent link="rgb_camera_link"/>
+      <child link="depth_camera_link_optical_frame"/>
     </joint>
     <gazebo reference="rgb_camera_link_optical_frame">
@@ -229,4 +233,60 @@
      </sensor>
     </gazebo>
+    <gazebo reference="segmentation_camera_link_optical_frame">
+     <sensor name="segmentation_camera" type="segmentation">
+        <camera>
+            <segmentation_type>instance</segmentation_type>
+            <horizontal_fov>1.047</horizontal_fov>
+            <image>
+                <width>320</width>
+                <height>240</height>
+            </image>
+            <clip>
+                <near>0.1</near>
+                <far>100</far>
+            </clip>
+        </camera>
+        <always_on>1</always_on>
+        <update_rate>30</update_rate>
+        <visualize>true</visualize>
+        <topic>segmentation</topic>
+     </sensor>
+    </gazebo>
+    <gazebo reference="depth_camera_link_optical_frame">
+     <sensor name="depth_camera1" type="depth_camera">
+        <camera>
+            <segmentation_type>instance</segmentation_type>
+            <horizontal_fov>1.047</horizontal_fov>
+            <image>
+                <width>256</width>
+                <height>256</height>
+            </image>
+            <clip>
+                <near>0.1</near>
+                <far>100</far>
+            </clip>
+        </camera>
+        <always_on>1</always_on>
+        <update_rate>30</update_rate>
+        <visualize>true</visualize>
+        <topic>depth_camera</topic>
+     </sensor>
+    </gazebo>
+    <gazebo reference="right_caster_wheel">
+     <mu1>0.001</mu1>
+     <mu2>0.001</mu2>
+    </gazebo>
+    <gazebo reference="left_caster_wheel">
+     <mu1>0.001</mu1>
+     <mu2>0.001</mu2>
+    </gazebo>
+    <gazebo reference="right_wheel">
+     <mu1>100.0</mu1>
+     <mu2>100.0</mu2>
+    </gazebo>
+    <gazebo reference="left_wheel">
+     <mu1>100.0</mu1>
+     <mu2>100.0</mu2>
+    </gazebo>
     <gazebo reference="base_left_caster_wheel">
      <preserveFixedJoint>true</preserveFixedJoint>
@@ -241,4 +301,10 @@
      <preserveFixedJoint>true</preserveFixedJoint>
     </gazebo>
+    <gazebo reference="segmentation_camera_link_optical_frame_joint">
+     <preserveFixedJoint>true</preserveFixedJoint>
+    </gazebo>
+    <gazebo reference="depth_camera_link_optical_frame_joint">
+     <preserveFixedJoint>true</preserveFixedJoint>
+    </gazebo>
     <gazebo reference="base_chassis_joint">
      <preserveFixedJoint>true</preserveFixedJoint>

Commit message: adding odom publishing bridge

File: rae_description/urdf/rae_gazebo.urdf.xacro (robot description, xacro)
@@ -16,5 +16,5 @@
     </gazebo>
     <link name="chassis">
-      <xacro:body mass="0.2" d="0.125" h="0.028" w="0.1256">
+      <xacro:body mass="0.360" d="0.125" h="0.028" w="0.1256">
           <origin xyz="0 0.014 0.0" rpy="0.0 0.0 0.0"/>
       </xacro:body>
@@ -45,6 +45,6 @@
         <origin rpy="1.57 0.0 1.57" xyz="0.0307 0.0 0.0" />
     </joint>
-    <link name="left_wheel">
-      <xacro:wheels mass="0.05" h="0.01" r="0.0125">
+   <!-- <link name="left_wheel">
+      <xacro:wheels mass="0.008" h="0.011" r="0.0119">
             <origin xyz="-0.005 0.0 0.0" rpy="0.0 0.0 0.0"/>
       </xacro:wheels>
@@ -61,7 +61,53 @@
         </geometry>
       </visual>
+    </link> -->
+    <link name="left_wheel">
+      <xacro:wheels mass="0.008" h="0.011" r="0.0119">
+            <origin xyz="0.0 0.0 -0.0055" rpy="0.0 0.0 0.0"/>
+      </xacro:wheels>
+      <collision>
+        <origin rpy="0.0 0.0 0.0" xyz="0.0 0.0 -0.0055"/>
+        <geometry>
+            <cylinder length="0.011" radius="0.0119"/>
+        </geometry>
+      </collision>
+      <visual>
+        <origin rpy="0.0 0.0 0.0" xyz="0.0 0.0 -0.0055"/>
+        <geometry>
+            <cylinder length="0.011" radius="0.0119"/>
+        </geometry>
+      </visual>
     </link>
     <link name="right_wheel">
-      <xacro:wheels mass="0.05" h="0.01" r="0.0125">
+      <xacro:wheels mass="0.008" h="0.011" r="0.0119">
+            <origin xyz="0.0 0.0 -0.0055" rpy="0.0 0.0 0.0"/>
+      </xacro:wheels>
+      <collision>
+        <origin rpy="0.0 0.0 0.0" xyz="0.0 0.0 -0.0055"/>
+        <geometry>
+            <cylinder length="0.011" radius="0.0119"/>
+        </geometry>
+      </collision>
+      <visual>
+        <origin rpy="0.0 0.0 0.0" xyz="0.0 0.0 -0.0055"/>
+        <geometry>
+            <cylinder length="0.011" radius="0.0119"/>
+        </geometry>
+      </visual>
+    </link>
+    <joint name='left_wheel_hinge' type='continuous'>
+      <origin rpy="1.57 0.0 0.00 " xyz="0.0 0.042 0.0052"/>
+      <child  link="left_wheel"/>
+      <parent link="base_frame"/>
+      <axis rpy="0 0 0" xyz="0 0 -1"/>
+    </joint>
+    <joint name='right_wheel_hinge' type='continuous'>
+      <origin rpy="-1.57 0.0 0.0 " xyz="0.0 -0.042 0.0052"/>
+      <child  link="right_wheel"/>
+      <parent link="base_frame"/>
+      <axis rpy="0 0 0" xyz="0 0 1"/>
+    </joint>
+   <!-- <link name="right_wheel">
+      <xacro:wheels mass="0.008" h="0.011" r="0.0119">
             <origin xyz="-0.005 0.0 0.0" rpy="0.0 0.0 0.0"/>
       </xacro:wheels>
@@ -78,6 +124,6 @@
         </geometry>
       </visual>
-    </link>
-    <joint name='left_wheel_hinge' type='continuous'>
+    </link> -->
+   <!-- <joint name='left_wheel_hinge' type='continuous'>
       <origin rpy="0.0 0.0 -1.57 " xyz="0.0 0.0427 0.0052"/>
       <child  link="left_wheel"/>
@@ -90,7 +136,7 @@
       <parent link="base_frame"/>
       <axis rpy="0 0 0" xyz="1 0 0"/>
-    </joint>
+    </joint>-->
     <link name="left_caster_wheel">
-      <xacro:caster_wheels mass="0.035" r="0.005">
+      <xacro:caster_wheels mass="0.008" r="0.005">
             <origin xyz="0.0 0.0 0.0" rpy="0.0 0.0 0.0"/>
       </xacro:caster_wheels>
@@ -122,5 +168,5 @@
     </joint>
     <link name="right_caster_wheel">
-      <xacro:caster_wheels mass="0.035" r="0.005">
+      <xacro:caster_wheels mass="0.008" r="0.005">
             <origin xyz="0.0 0.0 0.0" rpy="0.0 0.0 0.0"/>
       </xacro:caster_wheels>
@@ -155,9 +201,13 @@
                 filename="libignition-gazebo-diff-drive-system.so"
                 name="ignition::gazebo::systems::DiffDrive">
+                <odometry_frame>base_frame</odometry_frame>
+                <publish_odom>true</publish_odom>
+                <publish_odom_tf>true</publish_odom_tf>
+                <odom_topic>odom</odom_topic>
                 <left_joint>left_wheel_hinge</left_joint>
                 <right_joint>right_wheel_hinge</right_joint>
                 <wheel_separation>0.0854</wheel_separation>
                 <!-- check correct wheel radius when you come back to the task -->
-                <wheel_radius>0.0125</wheel_radius>
+                <wheel_radius>0.0119</wheel_radius>
                 <odom_publish_frequency>1</odom_publish_frequency>
                 <topic>cmd_vel</topic>
@@ -215,5 +265,5 @@
     </joint>
     <gazebo reference="rgb_camera_link_optical_frame">
-     <sensor name="camera" type="camera">
+     <sensor name="rgbd_camera" type="rgbd_camera">
         <camera>
             <horizontal_fov>1.047</horizontal_fov>

Commit message: getting rid of box at the front

File: rae_description/urdf/rae_gazebo.urdf.xacro (robot description, xacro)
@@ -80,7 +80,21 @@
     </link>
     <link name="right_wheel">
-      <xacro:wheels mass="0.008" h="0.011" r="0.0119">
+      <!-- <xacro:wheels mass="0.008" h="0.011" r="0.0119">
             <origin xyz="0.0 0.0 -0.0055" rpy="0.0 0.0 0.0"/>
-      </xacro:wheels>
+      </xacro:wheels> -->
+    <inertial>
+      <origin
+        xyz="-0.046973 0.00518 -0.03067"
+        rpy="0 0 0" />
+      <mass
+        value="0.008" />
+      <inertia
+        ixx="2.8106E-07"
+        ixy="-3.5503E-14"
+        ixz="-3.4849E-10"
+        iyy="2.0307E-07"
+        iyz="3.6705E-14"
+        izz="2.0323E-07" />
+    </inertial>
       <collision>
         <origin rpy="0.0 0.0 0.0" xyz="0.0 0.0 -0.0055"/>
@@ -221,5 +235,5 @@
           <origin xyz="0.0 0.0 0.0" rpy="0.0 0.0 0.0"/>
      </xacro:body>
-     <visual>
+     <!-- <visual>
         <geometry>
             <box size="0.010 0.03 0.03"/>
@@ -230,5 +244,5 @@
             <box size="0.010 0.03 0.03"/>
         </geometry>
-     </collision>
+     </collision> -->
     </link>
     <joint name="rgb_camera_joint" type="fixed">
@@ -253,5 +267,5 @@
     </link>
     <joint name="rgb_camera_link_optical_frame_joint" type="fixed">
-      <origin xyz="0.0051 0 0" rpy="-1.57 0.0 -1.57"/>
+      <origin xyz="0.0051 0 0" rpy="0.0 0.0 0.0"/>
       <parent link="rgb_camera_link"/>
       <child link="rgb_camera_link_optical_frame"/>
@@ -306,5 +320,5 @@
      </sensor>
     </gazebo>
-    <gazebo reference="depth_camera_link_optical_frame">
+    <!-- <gazebo reference="depth_camera_link_optical_frame">
      <sensor name="depth_camera1" type="depth_camera">
         <camera>
@@ -325,5 +339,5 @@
         <topic>depth_camera</topic>
      </sensor>
-    </gazebo>
+    </gazebo>  -->
     <gazebo reference="right_caster_wheel">
      <mu1>0.001</mu1>
