Commit message: Add initial setup for RGB and depth cameras

File: rae_description/urdf/camera.urdf.xacro (robot description, xacro)
@@ -30,22 +30,43 @@
     </joint>
     <gazebo reference="rgb_camera_link_optical_frame">
-        <sensor name="rgbd_camera" type="camera">
-            <camera>
-                <horizontal_fov>1.047</horizontal_fov>
-                <image>
-                    <width>320</width>
-                    <height>240</height>
-                </image>
-                <clip>
-                    <near>0.1</near>
-                    <far>100</far>
-                </clip>
-            </camera>
-            <ignition_frame_id>rgb_camera_link_optical_frame</ignition_frame_id>
-            <always_on>1</always_on>
-            <update_rate>30</update_rate>
-            <visualize>true</visualize>
-            <topic>/camera/image</topic>
-        </sensor>
+      <sensor type="camera" name="rgbd_camera">
+        <always_on>true</always_on>
+        <update_rate>30.0</update_rate>
+        <topic>/right/image_raw</topic>
+        <visualize>false</visualize>
+        <ignition_frame_id>rgb_camera_link_optical_frame</ignition_frame_id>
+        <horizontal_fov>${60.0/180.0*pi}</horizontal_fov>
+        <image>
+          <width>320</width>
+          <height>240</height>
+        </image>
+        <clip>
+          <near>0.1</near>
+          <far>100</far>
+        </clip>
+      </sensor>
+      <sensor type="depth_camera" name="rgb_camera_link_optical_frame">
+        <always_on>true</always_on>
+        <update_rate>30.0</update_rate>
+        <topic>/depth/image</topic>
+        <visualize>false</visualize>
+        <ignition_frame_id>rgb_camera_link_optical_frame</ignition_frame_id>
+        <camera>
+          <horizontal_fov>${60.0/180.0*pi}</horizontal_fov>
+          <image>
+            <width>320</width>
+            <height>240</height>
+          </image>
+          <clip>
+            <near>0.1</near>
+            <far>100</far>
+          </clip>
+          <noise>
+            <type>gaussian</type>
+            <mean>0.0</mean>
+            <stddev>0.01</stddev>
+          </noise>
+        </camera>
+      </sensor>
     </gazebo>
 </robot>

File: rae_description/urdf/rae.urdf.xacro (robot description, xacro)
@@ -299,3 +299,98 @@
   </joint>
   <xacro:rae_ros2_control sim_mode="$(arg sim_mode)"/>
+  <xacro:if value="$(arg sim_mode)">
+    <link name="rae_rgb_camera_sim_frame">
+      <xacro:body mass="0.00001" d="0.0000010" h="0.000003" w="0.00003">
+        <origin xyz="0.0 0.0 0.0" rpy="0.0 0.0 0.0"/>
+      </xacro:body>
+    </link>
+    <joint name="rae_rgb_camera_sim_frame_joint" type="fixed">
+      <origin xyz="0.0 0 0" rpy="1.57 -1.57 0.0"/>
+      <parent link="rae_rgb_camera_optical_frame"/>
+      <child link="rae_rgb_camera_sim_frame"/>
+    </joint>
+    <gazebo reference="rae_rgb_camera_sim_frame">
+      <sensor type="camera" name="rgbd_camera">
+        <always_on>true</always_on>
+        <update_rate>30.0</update_rate>
+        <topic>/right/image_raw</topic>
+        <ignition_frame_id>rae_rgb_camera_optical_frame</ignition_frame_id>
+        <horizontal_fov>${60.0/180.0*pi}</horizontal_fov>
+        <image>
+          <width>320</width>
+          <height>240</height>
+        </image>
+        <clip>
+          <near>0.1</near>
+          <far>100</far>
+        </clip>
+      </sensor>
+      <plugin filename="ignition-gazebo-sensors-system" name="ignition::gazebo::systems::Sensors">
+        <engine>ogre2</engine>
+      </plugin>
+    </gazebo>
+    <link name="rae_depth_camera_front_frame">
+      <xacro:body mass="0.00001" d="0.00001" h="0.000003" w="0.00001">
+        <origin xyz="0.0 0.0 0.0" rpy="0.0 0.0 0.0"/>
+      </xacro:body>
+    </link>
+    <joint name="rae_depth_camera_front_frame_joint" type="fixed">
+      <origin xyz="0.0 0.0 0.0" rpy="0.0 0.0 0.0"/>
+      <parent link="base_link"/>
+      <child link="rae_depth_camera_front_frame"/>
+    </joint>
+    <gazebo reference="rae_depth_camera_front_frame">
+      <sensor name="front_depth_camera" type="depth_camera">
+        <update_rate>15.0</update_rate>
+        <topic>/front/depth/image</topic>
+        <ignition_frame_id>rae_depth_camera_front_frame</ignition_frame_id>
+        <camera>
+          <horizontal_fov>${60.0/180.0*pi}</horizontal_fov>
+          <image>
+            <width>320</width>
+            <height>240</height>
+          </image>
+          <clip>
+            <near>0.1</near>
+            <far>100.0</far>
+          </clip>
+        </camera>
+      </sensor>
+      <plugin filename="ignition-gazebo-sensors-system" name="ignition::gazebo::systems::Sensors">
+        <engine>ogre2</engine>
+      </plugin>
+    </gazebo>
+    <link name="rae_depth_camera_rear_frame">
+      <xacro:body mass="0.00001" d="0.00001" h="0.00001" w="0.00001">
+        <origin xyz="0.0 0.0 0.0" rpy="0.0 0.0 0.0"/>
+      </xacro:body>
+    </link>
+    <joint name="rae_depth_camera_rear_frame_joint" type="fixed">
+      <origin xyz="0.0 0.0 0.0" rpy="0.0 0.0 ${pi}"/>
+      <parent link="base_link"/>
+      <child link="rae_depth_camera_rear_frame"/>
+    </joint>
+    <gazebo reference="rae_depth_camera_rear_frame">
+      <sensor name="rear_depth_camera" type="depth_camera">
+        <update_rate>15.0</update_rate>
+        <topic>/rear/depth/image</topic>
+        <vizualize>true</vizualize>
+        <ignition_frame_id>rae_depth_camera_rear_frame</ignition_frame_id>
+        <camera>
+          <horizontal_fov>${60.0/180.0*pi}</horizontal_fov>
+          <image>
+            <width>320</width>
+            <height>240</height>
+          </image>
+          <clip>
+            <near>0.1</near>
+            <far>100.0</far>
+          </clip>
+        </camera>
+      </sensor>
+      <plugin filename="ignition-gazebo-sensors-system" name="ignition::gazebo::systems::Sensors">
+        <engine>ogre2</engine>
+      </plugin>
+    </gazebo>
+  </xacro:if>
 </robot>
