Commit message: wip

File: rae_description/urdf/rae.urdf.xacro (robot description, xacro)
@@ -3,4 +3,6 @@
   xmlns:xacro="http://ros.org/wiki/xacro">
   <xacro:include filename="inertial_moment_calc.xacro"/>
+  <xacro:include filename="rae_gazebo.xacro"/>
+  <xacro:property name="deg_to_rad" value="0.01745329251994329577" />
   <link name="base_footprint"/>
   <joint name="dummy" type="fixed">
@@ -52,21 +54,4 @@
     <origin rpy="1.57 0.0 1.57" xyz="0.0307 0.0 0.0" />
   </joint>
-  <!-- <link name="left_wheel">
-      <xacro:wheels mass="0.008" h="0.011" r="0.0119">
-            <origin xyz="-0.005 0.0 0.0" rpy="0.0 0.0 0.0"/>
-      </xacro:wheels>
-      <collision>
-        <origin rpy="0.0 0.0 0.0" xyz="-0.0125 0.0 0.0"/>
-        <geometry>
-            <mesh filename="package://rae_description/urdf/models/Motor-wheel.stl" scale="1.0 1.0 1.0"/>
-        </geometry>
-      </collision>
-      <visual>
-        <origin rpy="0.0 0.0 0.0" xyz="-0.0125 0.0 0.0"/>
-        <geometry>
-            <mesh filename="package://rae_description/urdf/models/Motor-wheel.stl" scale="1.0 1.0 1.0"/>
-        </geometry>
-      </visual>
-    </link> -->
   <link name="left_wheel">
     <xacro:wheels mass="0.008" h="0.011" r="0.0119">
@@ -87,26 +72,21 @@
   </link>
   <link name="right_wheel">
-    <!-- <xacro:wheels mass="0.008" h="0.011" r="0.0119">
-            <origin xyz="0.0 0.0 -0.0055" rpy="0.0 0.0 0.0"/>
-      </xacro:wheels> -->
-    <inertial>
-      <origin xyz="-0.046973 0.00518 -0.03067" rpy="0 0 0" />
-      <mass value="0.008" />
-      <inertia ixx="2.8106E-07" ixy="-3.5503E-14" ixz="-3.4849E-10" iyy="2.0307E-07" iyz="3.6705E-14" izz="2.0323E-07" />
-    </inertial>
-    <collision>
-      <origin rpy="0.0 0.0 0.0" xyz="0.0 0.0 -0.0055"/>
-      <geometry>
-        <cylinder length="0.011" radius="0.0119"/>
-      </geometry>
-    </collision>
-    <visual>
-      <origin rpy="0.0 0.0 0.0" xyz="0.0 0.0 -0.0055"/>
-      <geometry>
-        <cylinder length="0.011" radius="0.0119"/>
-      </geometry>
-    </visual>
-  </link>
-  <joint name='left_wheel_hinge' type='continuous'>
+    <xacro:wheels mass="0.008" h="0.011" r="0.0119">
+      <origin xyz="0.0 0.0 -0.0055" rpy="0.0 0.0 0.0"/>
+    </xacro:wheels>
+    <collision>
+      <origin rpy="0.0 0.0 0.0" xyz="0.0 0.0 -0.0055"/>
+      <geometry>
+        <cylinder length="0.011" radius="0.0119"/>
+      </geometry>
+    </collision>
+    <visual>
+      <origin rpy="0.0 0.0 0.0" xyz="0.0 0.0 -0.0055"/>
+      <geometry>
+        <cylinder length="0.011" radius="0.0119"/>
+      </geometry>
+    </visual>
+  </link>
+  <joint name='left_wheel_joint' type='continuous'>
     <origin rpy="1.57 0.0 0.00 " xyz="0.0 0.042 0.0052"/>
     <child link="left_wheel"/>
@@ -114,5 +94,5 @@
     <axis rpy="0 0 0" xyz="0 0 -1"/>
   </joint>
-  <joint name='right_wheel_hinge' type='continuous'>
+  <joint name='right_wheel_joint' type='continuous'>
     <origin rpy="-1.57 0.0 0.0 " xyz="0.0 -0.042 0.0052"/>
     <child link="right_wheel"/>
@@ -120,33 +100,4 @@
     <axis rpy="0 0 0" xyz="0 0 1"/>
   </joint>
-  <!-- <link name="right_wheel">
-      <xacro:wheels mass="0.008" h="0.011" r="0.0119">
-            <origin xyz="-0.005 0.0 0.0" rpy="0.0 0.0 0.0"/>
-      </xacro:wheels>
-      <collision>
-        <origin rpy="0.0 0.0 0.0" xyz="-0.0125 0.0 0.0"/>
-        <geometry>
-            <mesh filename="package://rae_description/urdf/models/Motor-wheel.stl" scale="1.0 1.0 1.0"/>
-        </geometry>
-      </collision>
-      <visual>
-        <origin rpy="0.0 0.0 0.0" xyz="-0.0125 0.0 0.0"/>
-        <geometry>
-            <mesh filename="package://rae_description/urdf/models/Motor-wheel.stl" scale="1.0 1.0 1.0"/>
-        </geometry>
-      </visual>
-    </link> -->
-  <!-- <joint name='left_wheel_hinge' type='continuous'>
-      <origin rpy="0.0 0.0 -1.57 " xyz="0.0 0.0427 0.0052"/>
-      <child link="left_wheel"/>
-      <parent link="base_link"/>
-      <axis rpy="0 0 0" xyz="-1 0 0"/>
-    </joint>
-    <joint name='right_wheel_hinge' type='continuous'>
-      <origin rpy="0.0 0.0 1.57 " xyz="0.0 -0.0427 0.0052"/>
-      <child link="right_wheel"/>
-      <parent link="base_link"/>
-      <axis rpy="0 0 0" xyz="1 0 0"/>
-    </joint>-->
   <link name="left_caster_wheel">
     <xacro:caster_wheels mass="0.008" r="0.005">
@@ -209,36 +160,8 @@
     <origin rpy="0.0 0.0 0.0" xyz="0.0735 -0.0445 -0.001" />
   </joint>
-  <gazebo>
-    <plugin filename="libignition-gazebo-diff-drive-system.so" name="ignition::gazebo::systems::DiffDrive">
-      <frame_id>odom</frame_id>
-      <child_frame_id>base_footprint</child_frame_id>
-      <tf_topic>tf</tf_topic>
-      <publish_odom>true</publish_odom>
-      <publish_odom_tf>true</publish_odom_tf>
-      <publish_wheel_tf>true</publish_wheel_tf>
-      <odom_topic>odom</odom_topic>
-      <left_joint>left_wheel_hinge</left_joint>
-      <right_joint>right_wheel_hinge</right_joint>
-      <wheel_separation>0.0854</wheel_separation>
-      <!-- check correct wheel radius when you come back to the task -->
-      <wheel_radius>0.0119</wheel_radius>
-      <odom_publish_frequency>50</odom_publish_frequency>
-      <topic>cmd_vel</topic>
-    </plugin>
-  </gazebo>
   <link name="rgb_camera_link">
     <xacro:body mass="0.001" d="0.010" h="0.03" w="0.03">
       <origin xyz="0.0 0.0 0.0" rpy="0.0 0.0 0.0"/>
     </xacro:body>
-    <!-- <visual>
-        <geometry>
-            <box size="0.010 0.03 0.03"/>
-        </geometry>
-     </visual>
-     <collision>
-        <geometry>
-            <box size="0.010 0.03 0.03"/>
-        </geometry>
-     </collision> -->
   </link>
   <joint name="rgb_camera_joint" type="fixed">
@@ -277,101 +200,3 @@
     <child link="depth_camera_link_optical_frame"/>
   </joint>
-  <gazebo reference="rgb_camera_link_optical_frame">
-    <sensor name="rgbd_camera" type="rgbd_camera">
-      <camera>
-        <horizontal_fov>1.047</horizontal_fov>
-        <image>
-          <width>320</width>
-          <height>240</height>
-        </image>
-        <clip>
-          <near>0.1</near>
-          <far>100</far>
-        </clip>
-      </camera>
-      <ignition_frame_id>rgb_camera_link_optical_frame</ignition_frame_id>
-      <always_on>1</always_on>
-      <update_rate>30</update_rate>
-      <visualize>true</visualize>
-      <topic>camera</topic>
-    </sensor>
-  </gazebo>
-  <gazebo reference="segmentation_camera_link_optical_frame">
-    <sensor name="segmentation_camera" type="segmentation">
-      <camera>
-        <segmentation_type>instance</segmentation_type>
-        <horizontal_fov>1.047</horizontal_fov>
-        <image>
-          <width>320</width>
-          <height>240</height>
-        </image>
-        <clip>
-          <near>0.1</near>
-          <far>100</far>
-        </clip>
-      </camera>
-      <ignition_frame_id>segmentation_camera_link_optical_frame</ignition_frame_id>
-      <always_on>1</always_on>
-      <update_rate>30</update_rate>
-      <visualize>true</visualize>
-      <topic>segmentation</topic>
-    </sensor>
-  </gazebo>
-  <!-- <gazebo reference="depth_camera_link_optical_frame">
-     <sensor name="depth_camera1" type="depth_camera">
-        <camera>
-            <segmentation_type>instance</segmentation_type>
-            <horizontal_fov>1.047</horizontal_fov>
-            <image>
-                <width>256</width>
-                <height>256</height>
-            </image>
-            <clip>
-                <near>0.1</near>
-                <far>100</far>
-            </clip>
-        </camera>
-        <always_on>1</always_on>
-        <update_rate>30</update_rate>
-        <visualize>true</visualize>
-        <topic>depth_camera</topic>
-     </sensor>
-    </gazebo>  -->
-  <gazebo reference="right_caster_wheel">
-    <mu1>0.001</mu1>
-    <mu2>0.001</mu2>
-  </gazebo>
-  <gazebo reference="left_caster_wheel">
-    <mu1>0.001</mu1>
-    <mu2>0.001</mu2>
-  </gazebo>
-  <gazebo reference="right_wheel">
-    <mu1>100.0</mu1>
-    <mu2>100.0</mu2>
-  </gazebo>
-  <gazebo reference="left_wheel">
-    <mu1>100.0</mu1>
-    <mu2>100.0</mu2>
-  </gazebo>
-  <!-- <gazebo reference="base_left_caster_wheel">
-     <preserveFixedJoint>true</preserveFixedJoint>
-    </gazebo>
-    <gazebo reference="base_right_caster_wheel">
-     <preserveFixedJoint>true</preserveFixedJoint>
-    </gazebo>
-    <gazebo reference="rgb_camera_joint">
-     <preserveFixedJoint>true</preserveFixedJoint>
-    </gazebo>
-    <gazebo reference="rgb_camera_link_optical_frame_joint">
-     <preserveFixedJoint>true</preserveFixedJoint>
-    </gazebo>
-    <gazebo reference="segmentation_camera_link_optical_frame_joint">
-     <preserveFixedJoint>true</preserveFixedJoint>
-    </gazebo>
-    <gazebo reference="depth_camera_link_optical_frame_joint">
-     <preserveFixedJoint>true</preserveFixedJoint>
-    </gazebo>
-    <gazebo reference="base_chassis_joint">
-     <preserveFixedJoint>true</preserveFixedJoint>
-    </gazebo> -->
 </robot>

Commit message: updates for slam

File: rae_description/urdf/rae.urdf.xacro (robot description, xacro)
@@ -201,3 +201,13 @@
     <child link="depth_camera_link_optical_frame"/>
   </joint>
+  <link name="rae_right_camera_optical_frame">
+    <xacro:body mass="0.00001" d="0.0000010" h="0.000003" w="0.00003">
+      <origin xyz="0.0 0.0 0.0" rpy="0.0 0.0 0.0"/>
+    </xacro:body>
+  </link>
+  <joint name="rae_right_camera_optical_frame_joint" type="fixed">
+    <origin xyz="0.0051 0 0" rpy="0.0 0.0 0.0"/>
+    <parent link="rgb_camera_link"/>
+    <child link="rae_right_camera_optical_frame"/>
+  </joint>
 </robot>

Commit message: ROS 2 Control (#4)

File: rae_description/urdf/rae.urdf.xacro (robot description, xacro)
@@ -3,4 +3,7 @@
   xmlns:xacro="http://ros.org/wiki/xacro">
   <xacro:include filename="inertial_moment_calc.xacro"/>
+  <xacro:include filename="rae_gazebo.xacro"/>
+  <xacro:include filename="rae_control.xacro"/>
+  <xacro:property name="deg_to_rad" value="0.01745329251994329577" />
   <link name="base_footprint"/>
   <joint name="dummy" type="fixed">
@@ -52,21 +55,4 @@
     <origin rpy="1.57 0.0 1.57" xyz="0.0307 0.0 0.0" />
   </joint>
-  <!-- <link name="left_wheel">
-      <xacro:wheels mass="0.008" h="0.011" r="0.0119">
-            <origin xyz="-0.005 0.0 0.0" rpy="0.0 0.0 0.0"/>
-      </xacro:wheels>
-      <collision>
-        <origin rpy="0.0 0.0 0.0" xyz="-0.0125 0.0 0.0"/>
-        <geometry>
-            <mesh filename="package://rae_description/urdf/models/Motor-wheel.stl" scale="1.0 1.0 1.0"/>
-        </geometry>
-      </collision>
-      <visual>
-        <origin rpy="0.0 0.0 0.0" xyz="-0.0125 0.0 0.0"/>
-        <geometry>
-            <mesh filename="package://rae_description/urdf/models/Motor-wheel.stl" scale="1.0 1.0 1.0"/>
-        </geometry>
-      </visual>
-    </link> -->
   <link name="left_wheel">
     <xacro:wheels mass="0.008" h="0.011" r="0.0119">
@@ -87,26 +73,21 @@
   </link>
   <link name="right_wheel">
-    <!-- <xacro:wheels mass="0.008" h="0.011" r="0.0119">
-            <origin xyz="0.0 0.0 -0.0055" rpy="0.0 0.0 0.0"/>
-      </xacro:wheels> -->
-    <inertial>
-      <origin xyz="-0.046973 0.00518 -0.03067" rpy="0 0 0" />
-      <mass value="0.008" />
-      <inertia ixx="2.8106E-07" ixy="-3.5503E-14" ixz="-3.4849E-10" iyy="2.0307E-07" iyz="3.6705E-14" izz="2.0323E-07" />
-    </inertial>
-    <collision>
-      <origin rpy="0.0 0.0 0.0" xyz="0.0 0.0 -0.0055"/>
-      <geometry>
-        <cylinder length="0.011" radius="0.0119"/>
-      </geometry>
-    </collision>
-    <visual>
-      <origin rpy="0.0 0.0 0.0" xyz="0.0 0.0 -0.0055"/>
-      <geometry>
-        <cylinder length="0.011" radius="0.0119"/>
-      </geometry>
-    </visual>
-  </link>
-  <joint name='left_wheel_hinge' type='continuous'>
+    <xacro:wheels mass="0.008" h="0.011" r="0.0119">
+      <origin xyz="0.0 0.0 -0.0055" rpy="0.0 0.0 0.0"/>
+    </xacro:wheels>
+    <collision>
+      <origin rpy="0.0 0.0 0.0" xyz="0.0 0.0 -0.0055"/>
+      <geometry>
+        <cylinder length="0.011" radius="0.0119"/>
+      </geometry>
+    </collision>
+    <visual>
+      <origin rpy="0.0 0.0 0.0" xyz="0.0 0.0 -0.0055"/>
+      <geometry>
+        <cylinder length="0.011" radius="0.0119"/>
+      </geometry>
+    </visual>
+  </link>
+  <joint name='left_wheel_joint' type='continuous'>
     <origin rpy="1.57 0.0 0.00 " xyz="0.0 0.042 0.0052"/>
     <child link="left_wheel"/>
@@ -114,5 +95,5 @@
     <axis rpy="0 0 0" xyz="0 0 -1"/>
   </joint>
-  <joint name='right_wheel_hinge' type='continuous'>
+  <joint name='right_wheel_joint' type='continuous'>
     <origin rpy="-1.57 0.0 0.0 " xyz="0.0 -0.042 0.0052"/>
     <child link="right_wheel"/>
@@ -120,33 +101,4 @@
     <axis rpy="0 0 0" xyz="0 0 1"/>
   </joint>
-  <!-- <link name="right_wheel">
-      <xacro:wheels mass="0.008" h="0.011" r="0.0119">
-            <origin xyz="-0.005 0.0 0.0" rpy="0.0 0.0 0.0"/>
-      </xacro:wheels>
-      <collision>
-        <origin rpy="0.0 0.0 0.0" xyz="-0.0125 0.0 0.0"/>
-        <geometry>
-            <mesh filename="package://rae_description/urdf/models/Motor-wheel.stl" scale="1.0 1.0 1.0"/>
-        </geometry>
-      </collision>
-      <visual>
-        <origin rpy="0.0 0.0 0.0" xyz="-0.0125 0.0 0.0"/>
-        <geometry>
-            <mesh filename="package://rae_description/urdf/models/Motor-wheel.stl" scale="1.0 1.0 1.0"/>
-        </geometry>
-      </visual>
-    </link> -->
-  <!-- <joint name='left_wheel_hinge' type='continuous'>
-      <origin rpy="0.0 0.0 -1.57 " xyz="0.0 0.0427 0.0052"/>
-      <child link="left_wheel"/>
-      <parent link="base_link"/>
-      <axis rpy="0 0 0" xyz="-1 0 0"/>
-    </joint>
-    <joint name='right_wheel_hinge' type='continuous'>
-      <origin rpy="0.0 0.0 1.57 " xyz="0.0 -0.0427 0.0052"/>
-      <child link="right_wheel"/>
-      <parent link="base_link"/>
-      <axis rpy="0 0 0" xyz="1 0 0"/>
-    </joint>-->
   <link name="left_caster_wheel">
     <xacro:caster_wheels mass="0.008" r="0.005">
@@ -209,36 +161,8 @@
     <origin rpy="0.0 0.0 0.0" xyz="0.0735 -0.0445 -0.001" />
   </joint>
-  <gazebo>
-    <plugin filename="libignition-gazebo-diff-drive-system.so" name="ignition::gazebo::systems::DiffDrive">
-      <frame_id>odom</frame_id>
-      <child_frame_id>base_footprint</child_frame_id>
-      <tf_topic>tf</tf_topic>
-      <publish_odom>true</publish_odom>
-      <publish_odom_tf>true</publish_odom_tf>
-      <publish_wheel_tf>true</publish_wheel_tf>
-      <odom_topic>odom</odom_topic>
-      <left_joint>left_wheel_hinge</left_joint>
-      <right_joint>right_wheel_hinge</right_joint>
-      <wheel_separation>0.0854</wheel_separation>
-      <!-- check correct wheel radius when you come back to the task -->
-      <wheel_radius>0.0119</wheel_radius>
-      <odom_publish_frequency>50</odom_publish_frequency>
-      <topic>cmd_vel</topic>
-    </plugin>
-  </gazebo>
   <link name="rgb_camera_link">
     <xacro:body mass="0.001" d="0.010" h="0.03" w="0.03">
       <origin xyz="0.0 0.0 0.0" rpy="0.0 0.0 0.0"/>
     </xacro:body>
-    <!-- <visual>
-        <geometry>
-            <box size="0.010 0.03 0.03"/>
-        </geometry>
-     </visual>
-     <collision>
-        <geometry>
-            <box size="0.010 0.03 0.03"/>
-        </geometry>
-     </collision> -->
   </link>
   <joint name="rgb_camera_joint" type="fixed">
@@ -277,101 +201,3 @@
     <child link="depth_camera_link_optical_frame"/>
   </joint>
-  <gazebo reference="rgb_camera_link_optical_frame">
-    <sensor name="rgbd_camera" type="rgbd_camera">
-      <camera>
-        <horizontal_fov>1.047</horizontal_fov>
-        <image>
-          <width>320</width>
-          <height>240</height>
-        </image>
-        <clip>
-          <near>0.1</near>
-          <far>100</far>
-        </clip>
-      </camera>
-      <ignition_frame_id>rgb_camera_link_optical_frame</ignition_frame_id>
-      <always_on>1</always_on>
-      <update_rate>30</update_rate>
-      <visualize>true</visualize>
-      <topic>camera</topic>
-    </sensor>
-  </gazebo>
-  <gazebo reference="segmentation_camera_link_optical_frame">
-    <sensor name="segmentation_camera" type="segmentation">
-      <camera>
-        <segmentation_type>instance</segmentation_type>
-        <horizontal_fov>1.047</horizontal_fov>
-        <image>
-          <width>320</width>
-          <height>240</height>
-        </image>
-        <clip>
-          <near>0.1</near>
-          <far>100</far>
-        </clip>
-      </camera>
-      <ignition_frame_id>segmentation_camera_link_optical_frame</ignition_frame_id>
-      <always_on>1</always_on>
-      <update_rate>30</update_rate>
-      <visualize>true</visualize>
-      <topic>segmentation</topic>
-    </sensor>
-  </gazebo>
-  <!-- <gazebo reference="depth_camera_link_optical_frame">
-     <sensor name="depth_camera1" type="depth_camera">
-        <camera>
-            <segmentation_type>instance</segmentation_type>
-            <horizontal_fov>1.047</horizontal_fov>
-            <image>
-                <width>256</width>
-                <height>256</height>
-            </image>
-            <clip>
-                <near>0.1</near>
-                <far>100</far>
-            </clip>
-        </camera>
-        <always_on>1</always_on>
-        <update_rate>30</update_rate>
-        <visualize>true</visualize>
-        <topic>depth_camera</topic>
-     </sensor>
-    </gazebo>  -->
-  <gazebo reference="right_caster_wheel">
-    <mu1>0.001</mu1>
-    <mu2>0.001</mu2>
-  </gazebo>
-  <gazebo reference="left_caster_wheel">
-    <mu1>0.001</mu1>
-    <mu2>0.001</mu2>
-  </gazebo>
-  <gazebo reference="right_wheel">
-    <mu1>100.0</mu1>
-    <mu2>100.0</mu2>
-  </gazebo>
-  <gazebo reference="left_wheel">
-    <mu1>100.0</mu1>
-    <mu2>100.0</mu2>
-  </gazebo>
-  <!-- <gazebo reference="base_left_caster_wheel">
-     <preserveFixedJoint>true</preserveFixedJoint>
-    </gazebo>
-    <gazebo reference="base_right_caster_wheel">
-     <preserveFixedJoint>true</preserveFixedJoint>
-    </gazebo>
-    <gazebo reference="rgb_camera_joint">
-     <preserveFixedJoint>true</preserveFixedJoint>
-    </gazebo>
-    <gazebo reference="rgb_camera_link_optical_frame_joint">
-     <preserveFixedJoint>true</preserveFixedJoint>
-    </gazebo>
-    <gazebo reference="segmentation_camera_link_optical_frame_joint">
-     <preserveFixedJoint>true</preserveFixedJoint>
-    </gazebo>
-    <gazebo reference="depth_camera_link_optical_frame_joint">
-     <preserveFixedJoint>true</preserveFixedJoint>
-    </gazebo>
-    <gazebo reference="base_chassis_joint">
-     <preserveFixedJoint>true</preserveFixedJoint>
-    </gazebo> -->
 </robot>

Commit message: added cameras

File: rae_description/urdf/rae.urdf.xacro (robot description, xacro)
@@ -171,4 +171,84 @@
     <origin xyz="0.09 0.0 0.025" rpy="0 0 0"/>
   </joint>
+  <link name="a_camera_link">
+    <xacro:body mass="0.001" d="0.010" h="0.03" w="0.03">
+      <origin xyz="0.0 0.0 0.0" rpy="0.0 0.0 0.0"/>
+    </xacro:body>
+  </link>
+   <joint name="a_camera_joint" type="fixed">
+    <parent link="chassis"/>
+    <child link="a_camera_link"/>
+    <origin xyz="0.0375 0.0100195 0.0515282" rpy="-0.523599 0 0"/>
+  </joint>
+  <link name="a_camera_link_optical_frame">
+    <xacro:body mass="0.00001" d="0.0000010" h="0.000003" w="0.00003">
+      <origin xyz="0.0 0.0 0.0" rpy="0.0 0.0 0.0"/>
+    </xacro:body>
+  </link>
+  <joint name="a_camera_link_optical_frame_joint" type="fixed">
+    <origin xyz="0.0 0 0" rpy="0.0 -1.57 0.0"/>
+    <parent link="a_camera_link"/>
+    <child link="a_camera_link_optical_frame"/>
+  </joint>
+  <link name="b_camera_link">
+    <xacro:body mass="0.001" d="0.010" h="0.03" w="0.03">
+      <origin xyz="0.0 0.0 0.0" rpy="0.0 0.0 0.0"/>
+    </xacro:body>
+  </link>
+   <joint name="b_camera_joint" type="fixed">
+    <parent link="chassis"/>
+    <child link="b_camera_link"/>
+    <origin xyz="-0.0375 0.0100195 0.0515282" rpy="-0.523599 0 0"/>
+  </joint>
+  <link name="b_camera_link_optical_frame">
+    <xacro:body mass="0.00001" d="0.0000010" h="0.000003" w="0.00003">
+      <origin xyz="0.0 0.0 0.0" rpy="0.0 0.0 0.0"/>
+    </xacro:body>
+  </link>
+  <joint name="b_camera_link_optical_frame_joint" type="fixed">
+    <origin xyz="0.000 0 0" rpy="0.0 -1.57 0.0"/>
+    <parent link="b_camera_link"/>
+    <child link="b_camera_link_optical_frame"/>
+  </joint>
+  <link name="c_camera_link">
+    <xacro:body mass="0.001" d="0.010" h="0.03" w="0.03">
+      <origin xyz="0.0 0.0 0.0" rpy="0.0 0.0 0.0"/>
+    </xacro:body>
+  </link>
+   <joint name="c_camera_joint" type="fixed">
+    <parent link="chassis"/>
+    <child link="c_camera_link"/>
+    <origin xyz="-0.0375 0.0100195 -0.0515282" rpy="0.523599 0 0"/>
+  </joint>
+  <link name="c_camera_link_optical_frame">
+    <xacro:body mass="0.00001" d="0.0000010" h="0.000003" w="0.00003">
+      <origin xyz="0.0 0.0 0.0" rpy="0.0 0.0 0.0"/>
+    </xacro:body>
+  </link>
+  <joint name="c_camera_link_optical_frame_joint" type="fixed">
+    <origin xyz="0.000 0 0" rpy="0.0 1.57  0.0"/>
+    <parent link="c_camera_link"/>
+    <child link="c_camera_link_optical_frame"/>
+  </joint>
+  <link name="d_camera_link">
+    <xacro:body mass="0.001" d="0.010" h="0.03" w="0.03">
+      <origin xyz="0.0 0.0 0.0" rpy="0.0 0.0 0.0"/>
+    </xacro:body>
+  </link>
+   <joint name="d_camera_joint" type="fixed">
+    <parent link="chassis"/>
+    <child link="d_camera_link"/>
+    <origin xyz="0.0375 0.0100195 -0.0515282" rpy="0.523599 0 0"/>
+  </joint>
+  <link name="d_camera_link_optical_frame">
+    <xacro:body mass="0.00001" d="0.0000010" h="0.000003" w="0.00003">
+      <origin xyz="0.0 0.0 0.0" rpy="0.0 0.0 0.0"/>
+    </xacro:body>
+  </link>
+  <joint name="d_camera_link_optical_frame_joint" type="fixed">
+    <origin xyz="0.000 0 0" rpy="0.0 1.57 0.0"/>
+    <parent link="d_camera_link"/>
+    <child link="d_camera_link_optical_frame"/>
+  </joint>
   <link name="rgb_camera_link_optical_frame">
     <xacro:body mass="0.00001" d="0.0000010" h="0.000003" w="0.00003">

Commit message: fixing wheel rotation

File: rae_description/urdf/rae.urdf.xacro (robot description, xacro)
@@ -93,5 +93,5 @@
     <child link="left_wheel"/>
     <parent link="base_link"/>
-    <axis rpy="0 0 0" xyz="0 0 -1"/>
+    <axis rpy="0 0 0" xyz="0 0 1"/>
   </joint>
   <joint name='right_wheel_joint' type='continuous'>
@@ -99,5 +99,5 @@
     <child link="right_wheel"/>
     <parent link="base_link"/>
-    <axis rpy="0 0 0" xyz="0 0 1"/>
+    <axis rpy="0 0 0" xyz="0 0 -1"/>
   </joint>
   <link name="left_caster_wheel">

Commit message: lightweight model chassis

File: rae_description/urdf/rae.urdf.xacro (robot description, xacro)
@@ -38,5 +38,5 @@
       <origin rpy="0.0 0.0 0.0" xyz="0.0 0.0 0.0"/>
       <geometry>
-        <mesh filename="package://rae_description/urdf/models/RAE.stl" scale="1.0 1.0 1.0"/>
+        <mesh filename="package://rae_description/urdf/models/RAE-TOP-ASSY_0417.STL" scale="1.0 1.0 1.0"/>
       </geometry>
       <material name="mat">
