Commit message: optical coordinate frames set to be y front, z down, x right

File: rae_description/urdf/rae.urdf.xacro (robot description, xacro)
@@ -187,5 +187,5 @@
   </link>
   <joint name="a_camera_link_optical_frame_joint" type="fixed">
-    <origin xyz="0.0 0 0" rpy="0.0 -1.57 0.0"/>
+    <origin xyz="0.0 0 0" rpy="3.14 3.14 0.0"/>
     <parent link="a_camera_link"/>
     <child link="a_camera_link_optical_frame"/>
@@ -207,5 +207,5 @@
   </link>
   <joint name="b_camera_link_optical_frame_joint" type="fixed">
-    <origin xyz="0.000 0 0" rpy="0.0 -1.57 0.0"/>
+    <origin xyz="0.000 0 0" rpy="3.14 3.14 0.0"/>
     <parent link="b_camera_link"/>
     <child link="b_camera_link_optical_frame"/>
@@ -227,5 +227,5 @@
   </link>
   <joint name="c_camera_link_optical_frame_joint" type="fixed">
-    <origin xyz="0.000 0 0" rpy="0.0 1.57  0.0"/>
+    <origin xyz="0.000 0 0" rpy="3.14 0.0 0.0"/>
     <parent link="c_camera_link"/>
     <child link="c_camera_link_optical_frame"/>
@@ -247,5 +247,5 @@
   </link>
   <joint name="d_camera_link_optical_frame_joint" type="fixed">
-    <origin xyz="0.000 0 0" rpy="0.0 1.57 0.0"/>
+    <origin xyz="0.000 0 0" rpy="3.14 0.0 0.0"/>
     <parent link="d_camera_link"/>
     <child link="d_camera_link_optical_frame"/>

Commit message: updated slam, added temp depthscan conv

File: rae_description/urdf/rae.urdf.xacro (robot description, xacro)
@@ -207,6 +207,6 @@
   </link>
   <joint name="rae_right_camera_optical_frame_joint" type="fixed">
-    <origin xyz="0.0051 0 0" rpy="0.0 0.0 0.0"/>
-    <parent link="rgb_camera_link"/>
+    <origin xyz="0.051 0.064 0.01" rpy="-1.0472 0 -1.57"/>
+    <parent link="base_link"/>
     <child link="rae_right_camera_optical_frame"/>
   </joint>

Commit message: renaming cameras

File: rae_description/urdf/rae.urdf.xacro (robot description, xacro)
@@ -36,5 +36,5 @@
     </collision>
     <visual>
-      <origin rpy="0.0 0.0 0.0" xyz="0.0 0.0 0.0"/>
+      <origin rpy="0.0 3.14 0.0" xyz="0.0 0.0 0.0"/>
       <geometry>
         <mesh filename="package://rae_description/urdf/models/RAE-TOP-ASSY_0417.STL" scale="1.0 1.0 1.0"/>
@@ -53,5 +53,5 @@
     <parent link="base_link"/>
     <child link="chassis"/>
-    <origin rpy="1.57 0.0 1.57" xyz="0.0307 0.0 0.0" />
+    <origin rpy="1.57 0.0 1.57" xyz="-0.0307 0.0 0.0" />
   </joint>
   <link name="left_wheel">
@@ -93,5 +93,5 @@
     <child link="left_wheel"/>
     <parent link="base_link"/>
-    <axis rpy="0 0 0" xyz="0 0 1"/>
+    <axis rpy="0 0 0" xyz="0 0 -1"/>
   </joint>
   <joint name='right_wheel_joint' type='continuous'>
@@ -99,5 +99,5 @@
     <child link="right_wheel"/>
     <parent link="base_link"/>
-    <axis rpy="0 0 0" xyz="0 0 -1"/>
+    <axis rpy="0 0 0" xyz="0 0 1"/>
   </joint>
   <link name="left_caster_wheel">
@@ -129,5 +129,5 @@
     <parent link="base_link"/>
     <child link="left_caster_wheel"/>
-    <origin rpy="0.0 0.0 0.0" xyz="0.0735 0.0445 -0.001" />
+    <origin rpy="0.0 0.0 0.0" xyz="-0.0735 0.0445 -0.001" />
   </joint>
   <link name="right_caster_wheel">
@@ -159,5 +159,5 @@
     <parent link="base_link"/>
     <child link="right_caster_wheel"/>
-    <origin rpy="0.0 0.0 0.0" xyz="0.0735 -0.0445 -0.001" />
+    <origin rpy="0.0 0.0 0.0" xyz="-0.0735 -0.0445 -0.001" />
   </joint>
   <link name="rgb_camera_link">
@@ -167,87 +167,87 @@
   </link>
   <joint name="rgb_camera_joint" type="fixed">
-    <parent link="base_link"/>
+    <parent link="chassis"/>
     <child link="rgb_camera_link"/>
-    <origin xyz="0.09 0.0 0.025" rpy="0 0 0"/>
-  </joint>
-  <link name="a_camera_link">
-    <xacro:body mass="0.001" d="0.010" h="0.03" w="0.03">
-      <origin xyz="0.0 0.0 0.0" rpy="0.0 0.0 0.0"/>
-    </xacro:body>
-  </link>
-   <joint name="a_camera_joint" type="fixed">
-    <parent link="chassis"/>
-    <child link="a_camera_link"/>
+    <origin xyz="-0.025 0.0101195 0.0517014" rpy="-0.523599 0 0"/>
+  </joint>
+  <link name="left_front_camera_link">
+    <xacro:body mass="0.001" d="0.010" h="0.03" w="0.03">
+      <origin xyz="0.0 0.0 0.0" rpy="0.0 0.0 0.0"/>
+    </xacro:body>
+  </link>
+   <joint name="left_front_camera_joint" type="fixed">
+    <parent link="chassis"/>
+    <child link="left_front_camera_link"/>
     <origin xyz="0.0375 0.0100195 0.0515282" rpy="-0.523599 0 0"/>
   </joint>
-  <link name="a_camera_link_optical_frame">
-    <xacro:body mass="0.00001" d="0.0000010" h="0.000003" w="0.00003">
-      <origin xyz="0.0 0.0 0.0" rpy="0.0 0.0 0.0"/>
-    </xacro:body>
-  </link>
-  <joint name="a_camera_link_optical_frame_joint" type="fixed">
+  <link name="left_front_camera_link_optical_frame">
+    <xacro:body mass="0.00001" d="0.0000010" h="0.000003" w="0.00003">
+      <origin xyz="0.0 0.0 0.0" rpy="0.0 0.0 0.0"/>
+    </xacro:body>
+  </link>
+  <joint name="left_front_camera_link_optical_frame_joint" type="fixed">
     <origin xyz="0.0 0 0" rpy="3.14 3.14 0.0"/>
-    <parent link="a_camera_link"/>
-    <child link="a_camera_link_optical_frame"/>
-  </joint>
-  <link name="b_camera_link">
-    <xacro:body mass="0.001" d="0.010" h="0.03" w="0.03">
-      <origin xyz="0.0 0.0 0.0" rpy="0.0 0.0 0.0"/>
-    </xacro:body>
-  </link>
-   <joint name="b_camera_joint" type="fixed">
-    <parent link="chassis"/>
-    <child link="b_camera_link"/>
+    <parent link="left_front_camera_link"/>
+    <child link="left_front_camera_link_optical_frame"/>
+  </joint>
+  <link name="right_front_camera_link">
+    <xacro:body mass="0.001" d="0.010" h="0.03" w="0.03">
+      <origin xyz="0.0 0.0 0.0" rpy="0.0 0.0 0.0"/>
+    </xacro:body>
+  </link>
+   <joint name="right_front_camera_joint" type="fixed">
+    <parent link="chassis"/>
+    <child link="right_front_camera_link"/>
     <origin xyz="-0.0375 0.0100195 0.0515282" rpy="-0.523599 0 0"/>
   </joint>
-  <link name="b_camera_link_optical_frame">
-    <xacro:body mass="0.00001" d="0.0000010" h="0.000003" w="0.00003">
-      <origin xyz="0.0 0.0 0.0" rpy="0.0 0.0 0.0"/>
-    </xacro:body>
-  </link>
-  <joint name="b_camera_link_optical_frame_joint" type="fixed">
+  <link name="right_front_camera_link_optical_frame">
+    <xacro:body mass="0.00001" d="0.0000010" h="0.000003" w="0.00003">
+      <origin xyz="0.0 0.0 0.0" rpy="0.0 0.0 0.0"/>
+    </xacro:body>
+  </link>
+  <joint name="right_front_camera_link_optical_frame_joint" type="fixed">
     <origin xyz="0.000 0 0" rpy="3.14 3.14 0.0"/>
-    <parent link="b_camera_link"/>
-    <child link="b_camera_link_optical_frame"/>
-  </joint>
-  <link name="c_camera_link">
-    <xacro:body mass="0.001" d="0.010" h="0.03" w="0.03">
-      <origin xyz="0.0 0.0 0.0" rpy="0.0 0.0 0.0"/>
-    </xacro:body>
-  </link>
-   <joint name="c_camera_joint" type="fixed">
-    <parent link="chassis"/>
-    <child link="c_camera_link"/>
+    <parent link="right_front_camera_link"/>
+    <child link="right_front_camera_link_optical_frame"/>
+  </joint>
+  <link name="right_back_camera_link">
+    <xacro:body mass="0.001" d="0.010" h="0.03" w="0.03">
+      <origin xyz="0.0 0.0 0.0" rpy="0.0 0.0 0.0"/>
+    </xacro:body>
+  </link>
+   <joint name="right_back_camera_joint" type="fixed">
+    <parent link="chassis"/>
+    <child link="right_back_camera_link"/>
     <origin xyz="-0.0375 0.0100195 -0.0515282" rpy="0.523599 0 0"/>
   </joint>
-  <link name="c_camera_link_optical_frame">
-    <xacro:body mass="0.00001" d="0.0000010" h="0.000003" w="0.00003">
-      <origin xyz="0.0 0.0 0.0" rpy="0.0 0.0 0.0"/>
-    </xacro:body>
-  </link>
-  <joint name="c_camera_link_optical_frame_joint" type="fixed">
+  <link name="right_back_camera_link_optical_frame">
+    <xacro:body mass="0.00001" d="0.0000010" h="0.000003" w="0.00003">
+      <origin xyz="0.0 0.0 0.0" rpy="0.0 0.0 0.0"/>
+    </xacro:body>
+  </link>
+  <joint name="right_back_camera_link_optical_frame_joint" type="fixed">
     <origin xyz="0.000 0 0" rpy="3.14 0.0 0.0"/>
-    <parent link="c_camera_link"/>
-    <child link="c_camera_link_optical_frame"/>
-  </joint>
-  <link name="d_camera_link">
-    <xacro:body mass="0.001" d="0.010" h="0.03" w="0.03">
-      <origin xyz="0.0 0.0 0.0" rpy="0.0 0.0 0.0"/>
-    </xacro:body>
-  </link>
-   <joint name="d_camera_joint" type="fixed">
-    <parent link="chassis"/>
-    <child link="d_camera_link"/>
+    <parent link="right_back_camera_link"/>
+    <child link="right_back_camera_link_optical_frame"/>
+  </joint>
+  <link name="left_back_camera_link">
+    <xacro:body mass="0.001" d="0.010" h="0.03" w="0.03">
+      <origin xyz="0.0 0.0 0.0" rpy="0.0 0.0 0.0"/>
+    </xacro:body>
+  </link>
+   <joint name="left_back_camera_joint" type="fixed">
+    <parent link="chassis"/>
+    <child link="left_back_camera_link"/>
     <origin xyz="0.0375 0.0100195 -0.0515282" rpy="0.523599 0 0"/>
   </joint>
-  <link name="d_camera_link_optical_frame">
-    <xacro:body mass="0.00001" d="0.0000010" h="0.000003" w="0.00003">
-      <origin xyz="0.0 0.0 0.0" rpy="0.0 0.0 0.0"/>
-    </xacro:body>
-  </link>
-  <joint name="d_camera_link_optical_frame_joint" type="fixed">
+  <link name="left_back_camera_link_optical_frame">
+    <xacro:body mass="0.00001" d="0.0000010" h="0.000003" w="0.00003">
+      <origin xyz="0.0 0.0 0.0" rpy="0.0 0.0 0.0"/>
+    </xacro:body>
+  </link>
+  <joint name="left_back_camera_link_optical_frame_joint" type="fixed">
     <origin xyz="0.000 0 0" rpy="3.14 0.0 0.0"/>
-    <parent link="d_camera_link"/>
-    <child link="d_camera_link_optical_frame"/>
+    <parent link="left_back_camera_link"/>
+    <child link="left_back_camera_link_optical_frame"/>
   </joint>
   <link name="rgb_camera_link_optical_frame">
@@ -267,5 +267,5 @@
   </link>
   <joint name="rgb_camera_link_optical_frame_joint" type="fixed">
-    <origin xyz="0.0051 0 0" rpy="0.0 0.0 0.0"/>
+    <origin xyz="0.0051 0 0" rpy="3.14 3.14 0.0"/>
     <parent link="rgb_camera_link"/>
     <child link="rgb_camera_link_optical_frame"/>

Commit message: Added camera frames (#7)
* added cameras

* fixing wheel rotation

* lightweight model chassis

* optical coordinate frames set to be y front, z down, x right

* renaming cameras

---------

Co-authored-by: Danilo Pejovic <pejovicdanilo@outlook.com>

File: rae_description/urdf/rae.urdf.xacro (robot description, xacro)
@@ -36,7 +36,7 @@
     </collision>
     <visual>
-      <origin rpy="0.0 0.0 0.0" xyz="0.0 0.0 0.0"/>
-      <geometry>
-        <mesh filename="package://rae_description/urdf/models/RAE.stl" scale="1.0 1.0 1.0"/>
+      <origin rpy="0.0 3.14 0.0" xyz="0.0 0.0 0.0"/>
+      <geometry>
+        <mesh filename="package://rae_description/urdf/models/RAE-TOP-ASSY_0417.STL" scale="1.0 1.0 1.0"/>
       </geometry>
       <material name="mat">
@@ -53,5 +53,5 @@
     <parent link="base_link"/>
     <child link="chassis"/>
-    <origin rpy="1.57 0.0 1.57" xyz="0.0307 0.0 0.0" />
+    <origin rpy="1.57 0.0 1.57" xyz="-0.0307 0.0 0.0" />
   </joint>
   <link name="left_wheel">
@@ -129,5 +129,5 @@
     <parent link="base_link"/>
     <child link="left_caster_wheel"/>
-    <origin rpy="0.0 0.0 0.0" xyz="0.0735 0.0445 -0.001" />
+    <origin rpy="0.0 0.0 0.0" xyz="-0.0735 0.0445 -0.001" />
   </joint>
   <link name="right_caster_wheel">
@@ -159,5 +159,5 @@
     <parent link="base_link"/>
     <child link="right_caster_wheel"/>
-    <origin rpy="0.0 0.0 0.0" xyz="0.0735 -0.0445 -0.001" />
+    <origin rpy="0.0 0.0 0.0" xyz="-0.0735 -0.0445 -0.001" />
   </joint>
   <link name="rgb_camera_link">
@@ -167,7 +167,87 @@
   </link>
   <joint name="rgb_camera_joint" type="fixed">
-    <parent link="base_link"/>
+    <parent link="chassis"/>
     <child link="rgb_camera_link"/>
-    <origin xyz="0.09 0.0 0.025" rpy="0 0 0"/>
+    <origin xyz="-0.025 0.0101195 0.0517014" rpy="-0.523599 0 0"/>
+  </joint>
+  <link name="left_front_camera_link">
+    <xacro:body mass="0.001" d="0.010" h="0.03" w="0.03">
+      <origin xyz="0.0 0.0 0.0" rpy="0.0 0.0 0.0"/>
+    </xacro:body>
+  </link>
+   <joint name="left_front_camera_joint" type="fixed">
+    <parent link="chassis"/>
+    <child link="left_front_camera_link"/>
+    <origin xyz="0.0375 0.0100195 0.0515282" rpy="-0.523599 0 0"/>
+  </joint>
+  <link name="left_front_camera_link_optical_frame">
+    <xacro:body mass="0.00001" d="0.0000010" h="0.000003" w="0.00003">
+      <origin xyz="0.0 0.0 0.0" rpy="0.0 0.0 0.0"/>
+    </xacro:body>
+  </link>
+  <joint name="left_front_camera_link_optical_frame_joint" type="fixed">
+    <origin xyz="0.0 0 0" rpy="3.14 3.14 0.0"/>
+    <parent link="left_front_camera_link"/>
+    <child link="left_front_camera_link_optical_frame"/>
+  </joint>
+  <link name="right_front_camera_link">
+    <xacro:body mass="0.001" d="0.010" h="0.03" w="0.03">
+      <origin xyz="0.0 0.0 0.0" rpy="0.0 0.0 0.0"/>
+    </xacro:body>
+  </link>
+   <joint name="right_front_camera_joint" type="fixed">
+    <parent link="chassis"/>
+    <child link="right_front_camera_link"/>
+    <origin xyz="-0.0375 0.0100195 0.0515282" rpy="-0.523599 0 0"/>
+  </joint>
+  <link name="right_front_camera_link_optical_frame">
+    <xacro:body mass="0.00001" d="0.0000010" h="0.000003" w="0.00003">
+      <origin xyz="0.0 0.0 0.0" rpy="0.0 0.0 0.0"/>
+    </xacro:body>
+  </link>
+  <joint name="right_front_camera_link_optical_frame_joint" type="fixed">
+    <origin xyz="0.000 0 0" rpy="3.14 3.14 0.0"/>
+    <parent link="right_front_camera_link"/>
+    <child link="right_front_camera_link_optical_frame"/>
+  </joint>
+  <link name="right_back_camera_link">
+    <xacro:body mass="0.001" d="0.010" h="0.03" w="0.03">
+      <origin xyz="0.0 0.0 0.0" rpy="0.0 0.0 0.0"/>
+    </xacro:body>
+  </link>
+   <joint name="right_back_camera_joint" type="fixed">
+    <parent link="chassis"/>
+    <child link="right_back_camera_link"/>
+    <origin xyz="-0.0375 0.0100195 -0.0515282" rpy="0.523599 0 0"/>
+  </joint>
+  <link name="right_back_camera_link_optical_frame">
+    <xacro:body mass="0.00001" d="0.0000010" h="0.000003" w="0.00003">
+      <origin xyz="0.0 0.0 0.0" rpy="0.0 0.0 0.0"/>
+    </xacro:body>
+  </link>
+  <joint name="right_back_camera_link_optical_frame_joint" type="fixed">
+    <origin xyz="0.000 0 0" rpy="3.14 0.0 0.0"/>
+    <parent link="right_back_camera_link"/>
+    <child link="right_back_camera_link_optical_frame"/>
+  </joint>
+  <link name="left_back_camera_link">
+    <xacro:body mass="0.001" d="0.010" h="0.03" w="0.03">
+      <origin xyz="0.0 0.0 0.0" rpy="0.0 0.0 0.0"/>
+    </xacro:body>
+  </link>
+   <joint name="left_back_camera_joint" type="fixed">
+    <parent link="chassis"/>
+    <child link="left_back_camera_link"/>
+    <origin xyz="0.0375 0.0100195 -0.0515282" rpy="0.523599 0 0"/>
+  </joint>
+  <link name="left_back_camera_link_optical_frame">
+    <xacro:body mass="0.00001" d="0.0000010" h="0.000003" w="0.00003">
+      <origin xyz="0.0 0.0 0.0" rpy="0.0 0.0 0.0"/>
+    </xacro:body>
+  </link>
+  <joint name="left_back_camera_link_optical_frame_joint" type="fixed">
+    <origin xyz="0.000 0 0" rpy="3.14 0.0 0.0"/>
+    <parent link="left_back_camera_link"/>
+    <child link="left_back_camera_link_optical_frame"/>
   </joint>
   <link name="rgb_camera_link_optical_frame">
@@ -187,5 +267,5 @@
   </link>
   <joint name="rgb_camera_link_optical_frame_joint" type="fixed">
-    <origin xyz="0.0051 0 0" rpy="0.0 0.0 0.0"/>
+    <origin xyz="0.0051 0 0" rpy="3.14 3.14 0.0"/>
     <parent link="rgb_camera_link"/>
     <child link="rgb_camera_link_optical_frame"/>

Commit message: update launch files

File: rae_description/urdf/rae.urdf.xacro (robot description, xacro)
@@ -3,6 +3,6 @@
   xmlns:xacro="http://ros.org/wiki/xacro">
   <xacro:include filename="inertial_moment_calc.xacro"/>
-  <xacro:include filename="rae_gazebo.xacro"/>
-  <xacro:include filename="rae_control.xacro"/>
+  <!-- <xacro:include filename="rae_gazebo.xacro"/> -->
+  <xacro:include filename="rae_ros2_control.urdf.xacro"/>
   <xacro:property name="deg_to_rad" value="0.01745329251994329577" />
   <link name="base_footprint"/>
@@ -281,5 +281,5 @@
     <child link="depth_camera_link_optical_frame"/>
   </joint>
-  <link name="rae_right_camera_optical_frame">
+  <link name="rae_right_front_camera_optical_frame">
     <xacro:body mass="0.00001" d="0.0000010" h="0.000003" w="0.00003">
       <origin xyz="0.0 0.0 0.0" rpy="0.0 0.0 0.0"/>
@@ -289,5 +289,5 @@
     <origin xyz="0.051 0.064 0.01" rpy="-1.0472 0 -1.57"/>
     <parent link="base_link"/>
-    <child link="rae_right_camera_optical_frame"/>
+    <child link="rae_right_front_camera_optical_frame"/>
   </joint>
 </robot>

Commit message: wip rtabmap

File: rae_description/urdf/rae.urdf.xacro (robot description, xacro)
@@ -291,3 +291,13 @@
     <child link="rae_right_front_camera_optical_frame"/>
   </joint>
+    <link name="rae_left_front_camera_optical_frame">
+    <xacro:body mass="0.00001" d="0.0000010" h="0.000003" w="0.00003">
+      <origin xyz="0.0 0.0 0.0" rpy="0.0 0.0 0.0"/>
+    </xacro:body>
+  </link>
+  <joint name="rae_left_camera_optical_frame_joint" type="fixed">
+    <origin xyz="-0.051 0.064 0.01" rpy="-1.0472 0 -1.57"/>
+    <parent link="base_link"/>
+    <child link="rae_left_front_camera_optical_frame"/>
+  </joint>
 </robot>

Commit message: Slam depth update (#8)
* added cameras

* fixing wheel rotation

* Added description and gazebo packages

* lightweight model chassis

* add motor & encoder tests

* optical coordinate frames set to be y front, z down, x right

* updated slam, added temp depthscan conv

* Added rae_hw

* update to latest hw

* Added depthai-ros to the Dockerfile

* renaming cameras

* add camera example

* update depthimage

* add camera example

* add bringup dir

* add closed loop control

* update workflow

* change image

* update dockerfile

* add rosdep init

* typo

* add laserscan_kinect

* update launch files

* push image

* change ref

* change ref

* ref name

* head ref

* wip rtabmap

* add slam dependencies

* launch file reorganization

* update gz world

* update base image

* add cal.json

* update rosdep

* Update main.workflow.yaml

* add gst_bridge

* update dockerfile

* change to match repo name

* Adding relevant config files (#12)

* Adding relevant config files

* Update main.workflow.yaml

---------

Co-authored-by: Danilo Pejovic <pejovicdanilo@outlook.com>
Co-authored-by: Matej Hladky <mat.hladky@gmail.com>
Co-authored-by: Danilo Pejovic <115164734+danilo-pejovic@users.noreply.github.com>

File: rae_description/urdf/rae.urdf.xacro (robot description, xacro)
@@ -3,6 +3,6 @@
   xmlns:xacro="http://ros.org/wiki/xacro">
   <xacro:include filename="inertial_moment_calc.xacro"/>
-  <xacro:include filename="rae_gazebo.xacro"/>
-  <xacro:include filename="rae_control.xacro"/>
+  <!-- <xacro:include filename="rae_gazebo.xacro"/> -->
+  <xacro:include filename="rae_ros2_control.urdf.xacro"/>
   <xacro:property name="deg_to_rad" value="0.01745329251994329577" />
   <link name="base_footprint"/>
@@ -281,5 +281,5 @@
     <child link="depth_camera_link_optical_frame"/>
   </joint>
-  <link name="rae_right_camera_optical_frame">
+  <link name="rae_right_front_camera_optical_frame">
     <xacro:body mass="0.00001" d="0.0000010" h="0.000003" w="0.00003">
       <origin xyz="0.0 0.0 0.0" rpy="0.0 0.0 0.0"/>
@@ -287,7 +287,17 @@
   </link>
   <joint name="rae_right_camera_optical_frame_joint" type="fixed">
-    <origin xyz="0.0051 0 0" rpy="0.0 0.0 0.0"/>
-    <parent link="rgb_camera_link"/>
-    <child link="rae_right_camera_optical_frame"/>
+    <origin xyz="0.051 0.064 0.01" rpy="-1.0472 0 -1.57"/>
+    <parent link="base_link"/>
+    <child link="rae_right_front_camera_optical_frame"/>
+  </joint>
+    <link name="rae_left_front_camera_optical_frame">
+    <xacro:body mass="0.00001" d="0.0000010" h="0.000003" w="0.00003">
+      <origin xyz="0.0 0.0 0.0" rpy="0.0 0.0 0.0"/>
+    </xacro:body>
+  </link>
+  <joint name="rae_left_camera_optical_frame_joint" type="fixed">
+    <origin xyz="-0.051 0.064 0.01" rpy="-1.0472 0 -1.57"/>
+    <parent link="base_link"/>
+    <child link="rae_left_front_camera_optical_frame"/>
   </joint>
 </robot>
