Commit message: update urdf

File: rae_description/urdf/rae.urdf.xacro (robot description, xacro)
@@ -25,4 +25,14 @@
     </sensor>
   </gazebo>
+  <link name="base_link_back">
+    <xacro:body mass="0.00001" d="0.0000010" h="0.000003" w="0.00003">
+      <origin xyz="0.0 0.0 0.0" rpy="0.0 0.0 0"/>
+    </xacro:body>
+  </link>
+  <joint name="base_link_back_joint" type="fixed">
+    <parent link="base_link"/>
+    <child link="base_link_back"/>
+    <origin rpy="0 0.0 3.14" xyz="0.0 0.0 0.0" />
+  </joint>
   <link name="chassis">
     <xacro:body mass="0.360" d="0.125" h="0.028" w="0.1256">
@@ -161,143 +171,109 @@
     <origin rpy="0.0 0.0 0.0" xyz="-0.0735 -0.0445 -0.001" />
   </joint>
-  <link name="rgb_camera_link">
-    <xacro:body mass="0.001" d="0.010" h="0.03" w="0.03">
-      <origin xyz="0.0 0.0 0.0" rpy="0.0 0.0 0.0"/>
-    </xacro:body>
-  </link>
+  <link name="rae_rgb_camera_frame">
+    <xacro:body mass="0.001" d="0.010" h="0.03" w="0.03">
+      <origin xyz="0.0 0.0 0.0" rpy="0.0 0.0 0.0"/>
+    </xacro:body>
+  </link>
+  <link name="rae_rgb_camera_optical_frame">
+    <xacro:body mass="0.00001" d="0.0000010" h="0.000003" w="0.00003">
+      <origin xyz="0.0 0.0 0.0" rpy="0.0 0.0 0.0"/>
+    </xacro:body>
+  </link>
+  <joint name="rae_rgb_camera_optical_frame_joint" type="fixed">
+    <origin xyz="0.0051 0 0" rpy="3.14 3.14 0.0"/>
+    <parent link="rae_rgb_camera_frame"/>
+    <child link="rae_rgb_camera_optical_frame"/>
+  </joint>
   <joint name="rgb_camera_joint" type="fixed">
     <parent link="chassis"/>
-    <child link="rgb_camera_link"/>
+    <child link="rae_rgb_camera_frame"/>
     <origin xyz="-0.025 0.0101195 0.0517014" rpy="-0.523599 0 0"/>
   </joint>
-  <link name="left_front_camera_link">
-    <xacro:body mass="0.001" d="0.010" h="0.03" w="0.03">
-      <origin xyz="0.0 0.0 0.0" rpy="0.0 0.0 0.0"/>
-    </xacro:body>
-  </link>
-   <joint name="left_front_camera_joint" type="fixed">
-    <parent link="chassis"/>
-    <child link="left_front_camera_link"/>
+  <link name="rae_left_front_camera_frame">
+    <xacro:body mass="0.001" d="0.010" h="0.03" w="0.03">
+      <origin xyz="0.0 0.0 0.0" rpy="0.0 0.0 0.0"/>
+    </xacro:body>
+  </link>
+  <joint name="rae_left_front_camera_joint" type="fixed">
+    <parent link="chassis"/>
+    <child link="rae_left_front_camera_frame"/>
     <origin xyz="0.0375 0.0100195 0.0515282" rpy="-0.523599 0 0"/>
   </joint>
-  <link name="left_front_camera_link_optical_frame">
-    <xacro:body mass="0.00001" d="0.0000010" h="0.000003" w="0.00003">
-      <origin xyz="0.0 0.0 0.0" rpy="0.0 0.0 0.0"/>
-    </xacro:body>
-  </link>
-  <joint name="left_front_camera_link_optical_frame_joint" type="fixed">
+  <link name="rae_left_front_camera_optical_frame">
+    <xacro:body mass="0.00001" d="0.0000010" h="0.000003" w="0.00003">
+      <origin xyz="0.0 0.0 0.0" rpy="0.0 0.0 0.0"/>
+    </xacro:body>
+  </link>
+  <joint name="rae_left_front_camera_optical_frame_joint" type="fixed">
     <origin xyz="0.0 0 0" rpy="3.14 3.14 0.0"/>
-    <parent link="left_front_camera_link"/>
-    <child link="left_front_camera_link_optical_frame"/>
-  </joint>
-  <link name="right_front_camera_link">
-    <xacro:body mass="0.001" d="0.010" h="0.03" w="0.03">
-      <origin xyz="0.0 0.0 0.0" rpy="0.0 0.0 0.0"/>
-    </xacro:body>
-  </link>
-   <joint name="right_front_camera_joint" type="fixed">
-    <parent link="chassis"/>
-    <child link="right_front_camera_link"/>
+    <parent link="rae_left_front_camera_frame"/>
+    <child link="rae_left_front_camera_optical_frame"/>
+  </joint>
+  <link name="rae_right_front_camera_frame">
+    <xacro:body mass="0.001" d="0.010" h="0.03" w="0.03">
+      <origin xyz="0.0 0.0 0.0" rpy="0.0 0.0 0.0"/>
+    </xacro:body>
+  </link>
+  <joint name="rae_right_front_camera_joint" type="fixed">
+    <parent link="chassis"/>
+    <child link="rae_right_front_camera_frame"/>
     <origin xyz="-0.0375 0.0100195 0.0515282" rpy="-0.523599 0 0"/>
   </joint>
-  <link name="right_front_camera_link_optical_frame">
-    <xacro:body mass="0.00001" d="0.0000010" h="0.000003" w="0.00003">
-      <origin xyz="0.0 0.0 0.0" rpy="0.0 0.0 0.0"/>
-    </xacro:body>
-  </link>
-  <joint name="right_front_camera_link_optical_frame_joint" type="fixed">
+  <link name="rae_right_front_camera_optical_frame">
+    <xacro:body mass="0.00001" d="0.0000010" h="0.000003" w="0.00003">
+      <origin xyz="0.0 0.0 0.0" rpy="0.0 0.0 0.0"/>
+    </xacro:body>
+  </link>
+  <joint name="rae_right_front_camera_optical_frame_joint" type="fixed">
     <origin xyz="0.000 0 0" rpy="3.14 3.14 0.0"/>
-    <parent link="right_front_camera_link"/>
-    <child link="right_front_camera_link_optical_frame"/>
-  </joint>
-  <link name="right_back_camera_link">
-    <xacro:body mass="0.001" d="0.010" h="0.03" w="0.03">
-      <origin xyz="0.0 0.0 0.0" rpy="0.0 0.0 0.0"/>
-    </xacro:body>
-  </link>
-   <joint name="right_back_camera_joint" type="fixed">
-    <parent link="chassis"/>
-    <child link="right_back_camera_link"/>
+    <parent link="rae_right_front_camera_frame"/>
+    <child link="rae_right_front_camera_optical_frame"/>
+  </joint>
+  <link name="rae_right_back_camera_frame">
+    <xacro:body mass="0.001" d="0.010" h="0.03" w="0.03">
+      <origin xyz="0.0 0.0 0.0" rpy="0.0 0.0 0.0"/>
+    </xacro:body>
+  </link>
+  <joint name="rae_right_back_camera_joint" type="fixed">
+    <parent link="chassis"/>
+    <child link="rae_right_back_camera_frame"/>
     <origin xyz="-0.0375 0.0100195 -0.0515282" rpy="0.523599 0 0"/>
   </joint>
-  <link name="right_back_camera_link_optical_frame">
-    <xacro:body mass="0.00001" d="0.0000010" h="0.000003" w="0.00003">
-      <origin xyz="0.0 0.0 0.0" rpy="0.0 0.0 0.0"/>
-    </xacro:body>
-  </link>
-  <joint name="right_back_camera_link_optical_frame_joint" type="fixed">
+  <link name="rae_right_back_camera_optical_frame">
+    <xacro:body mass="0.00001" d="0.0000010" h="0.000003" w="0.00003">
+      <origin xyz="0.0 0.0 0.0" rpy="0.0 0.0 0.0"/>
+    </xacro:body>
+  </link>
+  <joint name="rae_right_back_camera_optical_frame_joint" type="fixed">
     <origin xyz="0.000 0 0" rpy="3.14 0.0 0.0"/>
-    <parent link="right_back_camera_link"/>
-    <child link="right_back_camera_link_optical_frame"/>
-  </joint>
-  <link name="left_back_camera_link">
-    <xacro:body mass="0.001" d="0.010" h="0.03" w="0.03">
-      <origin xyz="0.0 0.0 0.0" rpy="0.0 0.0 0.0"/>
-    </xacro:body>
-  </link>
-   <joint name="left_back_camera_joint" type="fixed">
-    <parent link="chassis"/>
-    <child link="left_back_camera_link"/>
+    <parent link="rae_right_back_camera_frame"/>
+    <child link="rae_right_back_camera_optical_frame"/>
+  </joint>
+  <link name="rae_left_back_camera_frame">
+    <xacro:body mass="0.001" d="0.010" h="0.03" w="0.03">
+      <origin xyz="0.0 0.0 0.0" rpy="0.0 0.0 0.0"/>
+    </xacro:body>
+  </link>
+  <joint name="rae_left_back_camera_joint" type="fixed">
+    <parent link="chassis"/>
+    <child link="rae_left_back_camera_frame"/>
     <origin xyz="0.0375 0.0100195 -0.0515282" rpy="0.523599 0 0"/>
   </joint>
-  <link name="left_back_camera_link_optical_frame">
-    <xacro:body mass="0.00001" d="0.0000010" h="0.000003" w="0.00003">
-      <origin xyz="0.0 0.0 0.0" rpy="0.0 0.0 0.0"/>
-    </xacro:body>
-  </link>
-  <joint name="left_back_camera_link_optical_frame_joint" type="fixed">
+  <link name="rae_left_back_camera_optical_frame">
+    <xacro:body mass="0.00001" d="0.0000010" h="0.000003" w="0.00003">
+      <origin xyz="0.0 0.0 0.0" rpy="0.0 0.0 0.0"/>
+    </xacro:body>
+  </link>
+  <joint name="rae_left_back_camera_optical_frame_joint" type="fixed">
     <origin xyz="0.000 0 0" rpy="3.14 0.0 0.0"/>
-    <parent link="left_back_camera_link"/>
-    <child link="left_back_camera_link_optical_frame"/>
-  </joint>
-  <link name="rgb_camera_link_optical_frame">
-    <xacro:body mass="0.00001" d="0.0000010" h="0.000003" w="0.00003">
-      <origin xyz="0.0 0.0 0.0" rpy="0.0 0.0 0.0"/>
-    </xacro:body>
-  </link>
-  <link name="segmentation_camera_link_optical_frame">
-    <xacro:body mass="0.00001" d="0.0000010" h="0.000003" w="0.00003">
-      <origin xyz="0.0 0.0 0.0" rpy="0.0 0.0 0.0"/>
-    </xacro:body>
-  </link>
-  <link name="depth_camera_link_optical_frame">
-    <xacro:body mass="0.00001" d="0.0000010" h="0.000003" w="0.00003">
-      <origin xyz="0.0 0.0 0.0" rpy="0.0 0.0 0.0"/>
-    </xacro:body>
-  </link>
-  <joint name="rgb_camera_link_optical_frame_joint" type="fixed">
-    <origin xyz="0.0051 0 0" rpy="3.14 3.14 0.0"/>
-    <parent link="rgb_camera_link"/>
-    <child link="rgb_camera_link_optical_frame"/>
-  </joint>
-  <joint name="segmentation_camera_link_optical_frame_joint" type="fixed">
-    <origin xyz="0.0051 0 0" rpy="0.0 0.0 0.0"/>
-    <parent link="rgb_camera_link"/>
-    <child link="segmentation_camera_link_optical_frame"/>
-  </joint>
-  <joint name="depth_camera_link_optical_frame_joint" type="fixed">
-    <origin xyz="0.0051 0 0" rpy="0.0 0.0 0.0"/>
-    <parent link="rgb_camera_link"/>
-    <child link="depth_camera_link_optical_frame"/>
-  </joint>
-  <link name="rae_right_front_camera_optical_frame">
-    <xacro:body mass="0.00001" d="0.0000010" h="0.000003" w="0.00003">
-      <origin xyz="0.0 0.0 0.0" rpy="0.0 0.0 0.0"/>
-    </xacro:body>
-  </link>
-  <joint name="rae_right_camera_optical_frame_joint" type="fixed">
-    <origin xyz="0.051 0.064 0.01" rpy="-1.0472 0 -1.57"/>
-    <parent link="base_link"/>
-    <child link="rae_right_front_camera_optical_frame"/>
-  </joint>
-    <link name="rae_left_front_camera_optical_frame">
-    <xacro:body mass="0.00001" d="0.0000010" h="0.000003" w="0.00003">
-      <origin xyz="0.0 0.0 0.0" rpy="0.0 0.0 0.0"/>
-    </xacro:body>
-  </link>
-  <joint name="rae_left_camera_optical_frame_joint" type="fixed">
-    <origin xyz="-0.051 0.064 0.01" rpy="-1.0472 0 -1.57"/>
-    <parent link="base_link"/>
-    <child link="rae_left_front_camera_optical_frame"/>
+    <parent link="rae_left_back_camera_frame"/>
+    <child link="rae_left_back_camera_optical_frame"/>
+  </joint>
+  <link name="rae_imu_frame"/>
+  <joint name="rae_imu_joint" type="fixed">
+    <origin xyz="0 0 0" rpy="0 0 0"/>
+    <parent link="base_link"/>
+    <child link="rae_imu_frame"/>
   </joint>
 </robot>

Commit message: update front camera names

File: rae_description/urdf/rae.urdf.xacro (robot description, xacro)
@@ -191,43 +191,43 @@
     <origin xyz="-0.025 0.0101195 0.0517014" rpy="-0.523599 0 0"/>
   </joint>
-  <link name="rae_left_front_camera_frame">
-    <xacro:body mass="0.001" d="0.010" h="0.03" w="0.03">
-      <origin xyz="0.0 0.0 0.0" rpy="0.0 0.0 0.0"/>
-    </xacro:body>
-  </link>
-  <joint name="rae_left_front_camera_joint" type="fixed">
-    <parent link="chassis"/>
-    <child link="rae_left_front_camera_frame"/>
+  <link name="rae_left_camera_frame">
+    <xacro:body mass="0.001" d="0.010" h="0.03" w="0.03">
+      <origin xyz="0.0 0.0 0.0" rpy="0.0 0.0 0.0"/>
+    </xacro:body>
+  </link>
+  <joint name="rae_left_camera_joint" type="fixed">
+    <parent link="chassis"/>
+    <child link="rae_left_camera_frame"/>
     <origin xyz="0.0375 0.0100195 0.0515282" rpy="-0.523599 0 0"/>
   </joint>
-  <link name="rae_left_front_camera_optical_frame">
-    <xacro:body mass="0.00001" d="0.0000010" h="0.000003" w="0.00003">
-      <origin xyz="0.0 0.0 0.0" rpy="0.0 0.0 0.0"/>
-    </xacro:body>
-  </link>
-  <joint name="rae_left_front_camera_optical_frame_joint" type="fixed">
+  <link name="rae_left_camera_optical_frame">
+    <xacro:body mass="0.00001" d="0.0000010" h="0.000003" w="0.00003">
+      <origin xyz="0.0 0.0 0.0" rpy="0.0 0.0 0.0"/>
+    </xacro:body>
+  </link>
+  <joint name="rae_left_camera_optical_frame_joint" type="fixed">
     <origin xyz="0.0 0 0" rpy="3.14 3.14 0.0"/>
-    <parent link="rae_left_front_camera_frame"/>
-    <child link="rae_left_front_camera_optical_frame"/>
-  </joint>
-  <link name="rae_right_front_camera_frame">
-    <xacro:body mass="0.001" d="0.010" h="0.03" w="0.03">
-      <origin xyz="0.0 0.0 0.0" rpy="0.0 0.0 0.0"/>
-    </xacro:body>
-  </link>
-  <joint name="rae_right_front_camera_joint" type="fixed">
-    <parent link="chassis"/>
-    <child link="rae_right_front_camera_frame"/>
+    <parent link="rae_left_camera_frame"/>
+    <child link="rae_left_camera_optical_frame"/>
+  </joint>
+  <link name="rae_right_camera_frame">
+    <xacro:body mass="0.001" d="0.010" h="0.03" w="0.03">
+      <origin xyz="0.0 0.0 0.0" rpy="0.0 0.0 0.0"/>
+    </xacro:body>
+  </link>
+  <joint name="rae_right_camera_joint" type="fixed">
+    <parent link="chassis"/>
+    <child link="rae_right_camera_frame"/>
     <origin xyz="-0.0375 0.0100195 0.0515282" rpy="-0.523599 0 0"/>
   </joint>
-  <link name="rae_right_front_camera_optical_frame">
-    <xacro:body mass="0.00001" d="0.0000010" h="0.000003" w="0.00003">
-      <origin xyz="0.0 0.0 0.0" rpy="0.0 0.0 0.0"/>
-    </xacro:body>
-  </link>
-  <joint name="rae_right_front_camera_optical_frame_joint" type="fixed">
+  <link name="rae_right_camera_optical_frame">
+    <xacro:body mass="0.00001" d="0.0000010" h="0.000003" w="0.00003">
+      <origin xyz="0.0 0.0 0.0" rpy="0.0 0.0 0.0"/>
+    </xacro:body>
+  </link>
+  <joint name="rae_right_camera_optical_frame_joint" type="fixed">
     <origin xyz="0.000 0 0" rpy="3.14 3.14 0.0"/>
-    <parent link="rae_right_front_camera_frame"/>
-    <child link="rae_right_front_camera_optical_frame"/>
+    <parent link="rae_right_camera_frame"/>
+    <child link="rae_right_camera_optical_frame"/>
   </joint>
   <link name="rae_right_back_camera_frame">

Commit message: Use ros2_control and add IMU to simulation

File: rae_description/urdf/rae.urdf.xacro (robot description, xacro)
@@ -2,6 +2,6 @@
 <robot name="rae"
   xmlns:xacro="http://ros.org/wiki/xacro">
+  <xacro:arg name="sim_mode" default="false" />
   <xacro:include filename="inertial_moment_calc.xacro"/>
-  <xacro:include filename="rae_gazebo_control.urdf.xacro"/>
   <xacro:include filename="rae_ros2_control.urdf.xacro"/>
   <xacro:property name="deg_to_rad" value="0.01745329251994329577" />
@@ -17,12 +17,21 @@
     </xacro:body>
   </link>
-  <gazebo reference="base_link">
-    <sensor name="imu_sensor" type="imu">
-      <always_on>1</always_on>
-      <update_rate>1</update_rate>
-      <visualize>true</visualize>
-      <topic>imu</topic>
-    </sensor>
-  </gazebo>
+  <xacro:if value="$(arg sim_mode)">
+    <gazebo reference="rae_imu_frame">
+      <sensor name="rae_imu_sensor" type="imu">
+        <always_on>1</always_on>
+        <update_rate>10.0</update_rate>
+        <visualize>true</visualize>
+        <topic>rae/imu/data</topic>
+        <frame_id>rae_imu_frame</frame_id>
+        <ignition_frame_id>rae_imu_frame</ignition_frame_id>
+      </sensor>
+    </gazebo>
+    <gazebo>
+      <plugin
+        filename="ignition-gazebo-imu-system" name="ignition::gazebo::systems::Imu">
+      </plugin>
+    </gazebo>
+  </xacro:if>
   <link name="base_link_back">
     <xacro:body mass="0.00001" d="0.0000010" h="0.000003" w="0.00003">
@@ -136,4 +145,10 @@
     </visual>
   </link>
+  <xacro:if value="$(arg sim_mode)">
+    <gazebo reference="left_caster_wheel">
+        <mu1>0.0001</mu1>
+        <mu2>0.0001</mu2>
+    </gazebo>
+  </xacro:if>
   <joint name="base_left_caster_wheel" type="fixed">
     <parent link="base_link"/>
@@ -166,4 +181,10 @@
     </visual>
   </link>
+  <xacro:if value="$(arg sim_mode)">
+    <gazebo reference="right_caster_wheel">
+        <mu1>0.0001</mu1>
+        <mu2>0.0001</mu2>
+    </gazebo>
+  </xacro:if>
   <joint name="base_right_caster_wheel" type="fixed">
     <parent link="base_link"/>
@@ -277,3 +298,4 @@
     <child link="rae_imu_frame"/>
   </joint>
+  <xacro:rae_ros2_control sim_mode="$(arg sim_mode)"/>
 </robot>

File: rae_description/urdf/rae_ros2_control.urdf.xacro (robot description, xacro)
@@ -2,49 +2,68 @@
 <robot name="rae"
   xmlns:xacro="http://ros.org/wiki/xacro">
-  <ros2_control name="RAE" type="system">
-    <hardware>
-      <plugin>rae_hw/RaeHW</plugin>
-      <param name="left_wheel_name">left_wheel_joint</param>
-      <param name="right_wheel_name">right_wheel_joint</param>
-      <param name="pwmName">/sys/class/pwm/pwmchip0</param>
-      <param name="pwmL">2</param>
-      <param name="pwmR">1</param>
-      <param name="phL">41</param>
-      <param name="phR">45</param>
-      <param name="enLA">42</param>
-      <param name="enLB">43</param>
-      <param name="enRA">46</param>
-      <param name="enRB">47</param>
-      <param name="encTicsPerRevL">756</param>
-      <param name="encTicsPerRevR">756</param>
-      <param name="maxVelL">32</param>
-      <param name="maxVelR">32</param>
-      <param name="closed_loopL">1</param>
-      <param name="PID_P_L">0.2</param>
-      <param name="PID_I_L">0.1</param>
-      <param name="PID_D_L">0.0005</param>
-      <param name="closed_loopR">1</param>
-      <param name="PID_P_R">0.2</param>
-      <param name="PID_I_R">0.1</param>
-      <param name="PID_D_R">0.0005</param>
-      <param name="loop_rate">30</param>
-      <param name="chip_name">gpiochip0</param>
-    </hardware>
-    <joint name="left_wheel_joint">
-      <command_interface name="velocity">
-        <param name="min">-1.68</param>
-        <param name="max">1.68</param>
-      </command_interface>
-      <state_interface name="velocity"/>
-      <state_interface name="position"/>
-    </joint>
-    <joint name="right_wheel_joint">
-      <command_interface name="velocity">
-        <param name="min">-1.68</param>
-        <param name="max">1.68</param>
-      </command_interface>
-      <state_interface name="velocity"/>
-      <state_interface name="position"/>
-    </joint>
-  </ros2_control>
+  <xacro:macro name="rae_ros2_control" params="sim_mode">
+    <ros2_control name="RAE" type="system">
+      <xacro:unless value="${sim_mode}">
+        <hardware>
+          <plugin>rae_hw/RaeHW</plugin>
+          <param name="left_wheel_name">left_wheel_joint</param>
+          <param name="right_wheel_name">right_wheel_joint</param>
+          <param name="pwmName">/sys/class/pwm/pwmchip0</param>
+          <param name="pwmL">2</param>
+          <param name="pwmR">1</param>
+          <param name="phL">41</param>
+          <param name="phR">45</param>
+          <param name="enLA">42</param>
+          <param name="enLB">43</param>
+          <param name="enRA">46</param>
+          <param name="enRB">47</param>
+          <param name="encTicsPerRevL">756</param>
+          <param name="encTicsPerRevR">756</param>
+          <param name="maxVelL">32</param>
+          <param name="maxVelR">32</param>
+          <param name="closed_loopL">1</param>
+          <param name="PID_P_L">0.2</param>
+          <param name="PID_I_L">0.1</param>
+          <param name="PID_D_L">0.0005</param>
+          <param name="closed_loopR">1</param>
+          <param name="PID_P_R">0.2</param>
+          <param name="PID_I_R">0.1</param>
+          <param name="PID_D_R">0.0005</param>
+          <param name="loop_rate">30</param>
+          <param name="chip_name">gpiochip0</param>
+        </hardware>
+      </xacro:unless>
+      <xacro:if value="${sim_mode}">
+        <hardware>
+          <plugin>ign_ros2_control/IgnitionSystem</plugin>
+        </hardware>
+      </xacro:if>
+      <joint name="left_wheel_joint">
+        <command_interface name="velocity">
+          <param name="min">-1.68</param>
+          <param name="max">1.68</param>
+        </command_interface>
+        <state_interface name="velocity"/>
+        <state_interface name="position"/>
+      </joint>
+      <joint name="right_wheel_joint">
+        <command_interface name="velocity">
+          <param name="min">-1.68</param>
+          <param name="max">1.68</param>
+        </command_interface>
+        <state_interface name="velocity"/>
+        <state_interface name="position"/>
+      </joint>
+    </ros2_control>
+    <xacro:if value="${sim_mode}">
+      <gazebo>
+        <plugin filename="ign_ros2_control-system" name="ign_ros2_control::IgnitionROS2ControlPlugin">
+          <parameters>$(find rae_hw)/config/controller.yaml</parameters>
+          <ros>
+            <remapping>/diff_controller/cmd_vel_unstamped:=/cmd_vel</remapping>
+          </ros>
+        </plugin>
+      </gazebo>
+    </xacro:if>
+  </xacro:macro>
 </robot>
