Commit message: Fix pointcloud and simtime for EKF

File: rae_description/urdf/rae.urdf.xacro (robot description, xacro)
@@ -210,5 +210,5 @@
     <parent link="chassis"/>
     <child link="rae_rgb_camera_frame"/>
-    <origin xyz="-0.025 0.0101195 0.0517014" rpy="-0.523599 0 0"/>
+    <origin xyz="-0.025 0.0101195 0.0517014" rpy="${-30.0/180*pi} 0 0"/>
   </joint>
   <link name="rae_left_camera_frame">
@@ -220,5 +220,5 @@
     <parent link="chassis"/>
     <child link="rae_left_camera_frame"/>
-    <origin xyz="0.0375 0.0100195 0.0515282" rpy="-0.523599 0 0"/>
+    <origin xyz="0.0375 0.0100195 0.0515282" rpy="${-30.0/180*pi} 0 0"/>
   </joint>
   <link name="rae_left_camera_optical_frame">
@@ -240,5 +240,5 @@
     <parent link="chassis"/>
     <child link="rae_right_camera_frame"/>
-    <origin xyz="-0.0375 0.0100195 0.0515282" rpy="-0.523599 0 0"/>
+    <origin xyz="-0.0375 0.0100195 0.0515282" rpy="${-30.0/180*pi} 0 0"/>
   </joint>
   <link name="rae_right_camera_optical_frame">
@@ -260,5 +260,5 @@
     <parent link="chassis"/>
     <child link="rae_right_back_camera_frame"/>
-    <origin xyz="-0.0375 0.0100195 -0.0515282" rpy="0.523599 0 0"/>
+    <origin xyz="-0.0375 0.0100195 -0.0515282" rpy="${30.0/180*pi} 0 0"/>
   </joint>
   <link name="rae_right_back_camera_optical_frame">
@@ -280,5 +280,5 @@
     <parent link="chassis"/>
     <child link="rae_left_back_camera_frame"/>
-    <origin xyz="0.0375 0.0100195 -0.0515282" rpy="0.523599 0 0"/>
+    <origin xyz="0.0375 0.0100195 -0.0515282" rpy="${30.0/180*pi} 0 0"/>
   </joint>
   <link name="rae_left_back_camera_optical_frame">
@@ -306,23 +306,30 @@
     </link>
     <joint name="rae_rgb_camera_sim_frame_joint" type="fixed">
-      <origin xyz="0.0 0 0" rpy="1.57 -1.57 0.0"/>
+      <origin xyz="0.0 0 0" rpy="${pi/2} ${-pi/2} 0.0"/>
       <parent link="rae_rgb_camera_optical_frame"/>
       <child link="rae_rgb_camera_sim_frame"/>
     </joint>
     <gazebo reference="rae_rgb_camera_sim_frame">
-      <sensor type="camera" name="rgbd_camera">
+      <sensor type="camera" name="rae_rgb_camera">
         <always_on>true</always_on>
         <update_rate>30.0</update_rate>
         <topic>/right/image_raw</topic>
         <ignition_frame_id>rae_rgb_camera_optical_frame</ignition_frame_id>
-        <horizontal_fov>${60.0/180.0*pi}</horizontal_fov>
-        <image>
-          <width>320</width>
-          <height>240</height>
-        </image>
-        <clip>
-          <near>0.1</near>
-          <far>100</far>
-        </clip>
+        <camera>
+          <horizontal_fov>${105.0/180.0*pi}</horizontal_fov>
+          <image>
+            <width>320</width>
+            <height>240</height>
+          </image>
+          <clip>
+            <near>0.1</near>
+            <far>100</far>
+          </clip>
+          <noise>
+            <type>gaussian</type>
+            <mean>0.0</mean>
+            <stddev>0.007</stddev>
+          </noise>
+        </camera>
       </sensor>
       <plugin filename="ignition-gazebo-sensors-system" name="ignition::gazebo::systems::Sensors">
@@ -336,5 +343,5 @@
     </link>
     <joint name="rae_depth_camera_front_frame_joint" type="fixed">
-      <origin xyz="0.0 0.0 0.0" rpy="0.0 0.0 0.0"/>
+      <origin xyz="${0.0208282} 0.0 0.0100195" rpy="0.0 ${-30.0/180*pi} 0.0"/>
       <parent link="base_link"/>
       <child link="rae_depth_camera_front_frame"/>
@@ -352,12 +359,9 @@
           </image>
           <clip>
-            <near>0.1</near>
-            <far>100.0</far>
+            <near>0.2</near>
+            <far>6.0</far>
           </clip>
         </camera>
       </sensor>
-      <plugin filename="ignition-gazebo-sensors-system" name="ignition::gazebo::systems::Sensors">
-        <engine>ogre2</engine>
-      </plugin>
     </gazebo>
     <link name="rae_depth_camera_rear_frame">
@@ -367,5 +371,5 @@
     </link>
     <joint name="rae_depth_camera_rear_frame_joint" type="fixed">
-      <origin xyz="0.0 0.0 0.0" rpy="0.0 0.0 ${pi}"/>
+      <origin xyz="${-0.0822282} 0.0 0.0100195" rpy="0.0 ${-30.0/180*pi} ${pi}"/>
       <parent link="base_link"/>
       <child link="rae_depth_camera_rear_frame"/>
@@ -384,12 +388,9 @@
           </image>
           <clip>
-            <near>0.1</near>
-            <far>100.0</far>
+            <near>0.2</near>
+            <far>6.0</far>
           </clip>
         </camera>
       </sensor>
-      <plugin filename="ignition-gazebo-sensors-system" name="ignition::gazebo::systems::Sensors">
-        <engine>ogre2</engine>
-      </plugin>
     </gazebo>
   </xacro:if>

Commit message: Unified topic names

File: rae_description/urdf/rae.urdf.xacro (robot description, xacro)
@@ -337,19 +337,19 @@
       </plugin>
     </gazebo>
-    <link name="rae_depth_camera_front_frame">
+    <link name="rae_stereo_front_frame">
       <xacro:body mass="0.00001" d="0.00001" h="0.000003" w="0.00001">
         <origin xyz="0.0 0.0 0.0" rpy="0.0 0.0 0.0"/>
       </xacro:body>
     </link>
-    <joint name="rae_depth_camera_front_frame_joint" type="fixed">
+    <joint name="rae_stereo_front_frame_joint" type="fixed">
       <origin xyz="${0.0208282} 0.0 0.0100195" rpy="0.0 ${-30.0/180*pi} 0.0"/>
       <parent link="base_link"/>
-      <child link="rae_depth_camera_front_frame"/>
+      <child link="rae_stereo_front_frame"/>
     </joint>
-    <gazebo reference="rae_depth_camera_front_frame">
+    <gazebo reference="rae_stereo_front_frame">
       <sensor name="front_depth_camera" type="depth_camera">
         <update_rate>15.0</update_rate>
-        <topic>/front/depth/image</topic>
-        <ignition_frame_id>rae_depth_camera_front_frame</ignition_frame_id>
+        <topic>/stereo_front/image_raw</topic>
+        <ignition_frame_id>rae_stereo_front_frame</ignition_frame_id>
         <camera>
           <horizontal_fov>${60.0/180.0*pi}</horizontal_fov>
@@ -365,20 +365,20 @@
       </sensor>
     </gazebo>
-    <link name="rae_depth_camera_rear_frame">
+    <link name="rae_stereo_rear_frame">
       <xacro:body mass="0.00001" d="0.00001" h="0.00001" w="0.00001">
         <origin xyz="0.0 0.0 0.0" rpy="0.0 0.0 0.0"/>
       </xacro:body>
     </link>
-    <joint name="rae_depth_camera_rear_frame_joint" type="fixed">
+    <joint name="rae_stereo_rear_frame_joint" type="fixed">
       <origin xyz="${-0.0822282} 0.0 0.0100195" rpy="0.0 ${-30.0/180*pi} ${pi}"/>
       <parent link="base_link"/>
-      <child link="rae_depth_camera_rear_frame"/>
+      <child link="rae_stereo_rear_frame"/>
     </joint>
-    <gazebo reference="rae_depth_camera_rear_frame">
+    <gazebo reference="rae_stereo_rear_frame">
       <sensor name="rear_depth_camera" type="depth_camera">
         <update_rate>15.0</update_rate>
-        <topic>/rear/depth/image</topic>
+        <topic>/stereo_back/image_raw</topic>
         <vizualize>true</vizualize>
-        <ignition_frame_id>rae_depth_camera_rear_frame</ignition_frame_id>
+        <ignition_frame_id>rae_stereo_rear_frame</ignition_frame_id>
         <camera>
           <horizontal_fov>${60.0/180.0*pi}</horizontal_fov>

Commit message: Unify topic names

File: rae_description/urdf/rae.urdf.xacro (robot description, xacro)
@@ -3,4 +3,5 @@
   xmlns:xacro="http://ros.org/wiki/xacro">
   <xacro:arg name="sim_mode" default="false" />
+  <xacro:arg name="namespace" default="" />
   <xacro:include filename="inertial_moment_calc.xacro"/>
   <xacro:include filename="rae_ros2_control.urdf.xacro"/>
@@ -23,5 +24,5 @@
         <update_rate>10.0</update_rate>
         <visualize>true</visualize>
-        <topic>rae/imu/data</topic>
+        <topic>/rae/imu/data</topic>
         <frame_id>rae_imu_frame</frame_id>
         <ignition_frame_id>rae_imu_frame</ignition_frame_id>
@@ -298,5 +299,5 @@
     <child link="rae_imu_frame"/>
   </joint>
-  <xacro:rae_ros2_control sim_mode="$(arg sim_mode)"/>
+  <xacro:rae_ros2_control sim_mode="$(arg sim_mode)" namespace="$(arg namespace)" />
   <xacro:if value="$(arg sim_mode)">
     <link name="rae_rgb_camera_sim_frame">
@@ -314,5 +315,5 @@
         <always_on>true</always_on>
         <update_rate>30.0</update_rate>
-        <topic>/right/image_raw</topic>
+        <topic>/rae/right/image_raw</topic>
         <ignition_frame_id>rae_rgb_camera_optical_frame</ignition_frame_id>
         <camera>
@@ -350,5 +351,5 @@
       <sensor name="front_depth_camera" type="depth_camera">
         <update_rate>15.0</update_rate>
-        <topic>/stereo_front/image_raw</topic>
+        <topic>/rae/stereo_front/image_raw</topic>
         <ignition_frame_id>rae_stereo_front_frame</ignition_frame_id>
         <camera>
@@ -378,5 +379,5 @@
       <sensor name="rear_depth_camera" type="depth_camera">
         <update_rate>15.0</update_rate>
-        <topic>/stereo_back/image_raw</topic>
+        <topic>/rae/stereo_back/image_raw</topic>
         <vizualize>true</vizualize>
         <ignition_frame_id>rae_stereo_rear_frame</ignition_frame_id>

File: rae_description/urdf/rae_ros2_control.urdf.xacro (robot description, xacro)
@@ -2,5 +2,5 @@
 <robot name="rae"
   xmlns:xacro="http://ros.org/wiki/xacro">
-  <xacro:macro name="rae_ros2_control" params="sim_mode">
+  <xacro:macro name="rae_ros2_control" params="sim_mode namespace">
     <ros2_control name="RAE" type="system">
       <xacro:unless value="${sim_mode}">
@@ -61,5 +61,6 @@
           <parameters>$(find rae_hw)/config/controller.yaml</parameters>
           <ros>
-            <remapping>/diff_controller/cmd_vel_unstamped:=/cmd_vel</remapping>
+            <namespace>${namespace}</namespace>
+            <remapping>diff_controller/cmd_vel_unstamped:=cmd_vel</remapping>
           </ros>
         </plugin>
